File: robot/Core.sch (KiCad schematic (older format))
At the start: 1 part

Commit message: added new core, changes to USBToUART
Parts:
- removed U?: ESP-12E, RF_Module:ESP-12E, symbol RF_Module:ESP-12E
- added U?: ESP32-WROOM-32, RF_Module:ESP32-WROOM-32, symbol RF_Module:ESP32-WROOM-32
Connections:
- net labels added: +3V3, GND
- wire segments 0 -> 2
Changed lines of the file:
@@
 $EndDescr
 $Comp
-L RF_Module:ESP-12E U?
-U 1 1 5D179708
-P 6050 3650
-F 0 "U?" H 6050 4631 50  0000 C CNN
-F 1 "ESP-12E" H 6050 4540 50  0000 C CNN
-F 2 "RF_Module:ESP-12E" H 6050 3650 50  0001 C CNN
-F 3 "http://wiki.ai-thinker.com/_media/esp8266/esp8266_series_modules_user_manual_v1.1.pdf" H 5700 3750 50  0001 C CNN
-	1    6050 3650
+L RF_Module:ESP32-WROOM-32 U?
+U 1 1 5D2E3B23
+P 5650 3950
+F 0 "U?" H 6050 5300 50  0000 C CNN
+F 1 "ESP32-WROOM-32" H 5150 5300 50  0000 C CNN
+F 2 "RF_Module:ESP32-WROOM-32" H 5650 2450 50  0001 C CNN
+F 3 "https://www.espressif.com/sites/default/files/documentation/esp32-wroom-32_datasheet_en.pdf" H 5350 4000 50  0001 C CNN
+	1    5650 3950
 	1    0    0    -1
 $EndComp
+$Comp
+L power:+3V3 #PWR?
+U 1 1 5D2E60B8
+P 5650 2250
+F 0 "#PWR?" H 5650 2100 50  0001 C CNN
+F 1 "+3V3" H 5665 2423 50  0000 C CNN
+F 2 "" H 5650 2250 50  0001 C CNN
+F 3 "" H 5650 2250 50  0001 C CNN
+	1    5650 2250
+	1    0    0    -1
+$EndComp
+Wire Wire Line
+	5650 2550 5650 2250
+$Comp
+L power:GND #PWR?
+U 1 1 5D2E6C58
+P 5650 5600
+F 0 "#PWR?" H 5650 5350 50  0001 C CNN
+F 1 "GND" H 5655 5427 50  0000 C CNN
+F 2 "" H 5650 5600 50  0001 C CNN
+F 3 "" H 5650 5600 50  0001 C CNN
+	1    5650 5600
+	1    0    0    -1
+$EndComp
+Wire Wire Line
+	5650 5350 5650 5600
 $EndSCHEMATC

Commit message: Object detection, reset
Parts:
- added C?: 1µ, symbol Device:C
- added R?: 10k, symbol Device:R
- added SW?: SW_Push, symbol Switch:SW_Push
Connections:
- net +3V3: now also R?.1
- net GND: now also C?.2, SW?.1
- net SDA_1: now reaches U?.21 (SDO/SD0)
- net SCL_1: now reaches U?.22 (SDI/SD1)
- net GPIO0: now reaches U?.25 (IO0)
- net EN: now reaches U?.3 (EN)
- net EN: now also C?.1, R?.2, SW?.2
- net RXD: now reaches U?.34 (RXD0/IO3)
- net TXD: now reaches U?.35 (TXD0/IO1)
Changed lines of the file:
@@
 $Descr A4 11693 8268
 encoding utf-8
-Sheet 3 4
+Sheet 3 5
 Title "Core"
 Date "2019-06-29"
@@
 Wire Wire Line
 	5650 5350 5650 5600
+Text HLabel 6450 2850 2    50   Input ~ 0
+TXD
+Text HLabel 6450 3050 2    50   Input ~ 0
+RXD
+Wire Wire Line
+	6250 2850 6450 2850
+Wire Wire Line
+	6250 3050 6450 3050
+Text HLabel 6450 2750 2    50   Input ~ 0
+GPIO0
+Text HLabel 3400 2750 0    50   Input ~ 0
+EN
+Wire Wire Line
+	3400 2750 3650 2750
+Wire Wire Line
+	6250 2750 6450 2750
+$Comp
+L Device:C C?
+U 1 1 5D6294B0
+P 4200 3050
+F 0 "C?" H 4315 3096 50  0000 L CNN
+F 1 "1µ" H 4315 3005 50  0000 L CNN
+F 2 "" H 4238 2900 50  0001 C CNN
+F 3 "~" H 4200 3050 50  0001 C CNN
+	1    4200 3050
+	1    0    0    -1
+$EndComp
+$Comp
+L Switch:SW_Push SW?
+U 1 1 5D62C889
+P 3650 3100
+F 0 "SW?" V 3750 2950 50  0000 C CNN
+F 1 "SW_Push" V 3600 2850 50  0000 C CNN
+F 2 "" H 3650 3300 50  0001 C CNN
+F 3 "~" H 3650 3300 50  0001 C CNN
+	1    3650 3100
+	0    -1   -1   0
+$EndComp
+$Comp
+L Device:R R?
+U 1 1 5D62DCB0
+P 3650 2450
+F 0 "R?" H 3720 2496 50  0000 L CNN
+F 1 "10k" H 3720 2405 50  0000 L CNN
+F 2 "" V 3580 2450 50  0001 C CNN
+F 3 "~" H 3650 2450 50  0001 C CNN
+	1    3650 2450
+	1    0    0    -1
+$EndComp
+$Comp
+L power:+3V3 #PWR?
+U 1 1 5D62E308
+P 3650 2200
+F 0 "#PWR?" H 3650 2050 50  0001 C CNN
+F 1 "+3V3" H 3665 2373 50  0000 C CNN
+F 2 "" H 3650 2200 50  0001 C CNN
+F 3 "" H 3650 2200 50  0001 C CNN
+	1    3650 2200
+	1    0    0    -1
+$EndComp
+$Comp
+L power:GND #PWR?
+U 1 1 5D62E7C3
+P 3650 3400
+F 0 "#PWR?" H 3650 3150 50  0001 C CNN
+F 1 "GND" H 3655 3227 50  0000 C CNN
+F 2 "" H 3650 3400 50  0001 C CNN
+F 3 "" H 3650 3400 50  0001 C CNN
+	1    3650 3400
+	1    0    0    -1
+$EndComp
+$Comp
+L power:GND #PWR?
+U 1 1 5D62EDF6
+P 4200 3300
+F 0 "#PWR?" H 4200 3050 50  0001 C CNN
+F 1 "GND" H 4205 3127 50  0000 C CNN
+F 2 "" H 4200 3300 50  0001 C CNN
+F 3 "" H 4200 3300 50  0001 C CNN
+	1    4200 3300
+	1    0    0    -1
+$EndComp
+Wire Wire Line
+	3650 2200 3650 2300
+Wire Wire Line
+	3650 2600 3650 2750
+Connection ~ 3650 2750
+Wire Wire Line
+	3650 2750 4200 2750
+Wire Wire Line
+	3650 2900 3650 2750
+Wire Wire Line
+	3650 3400 3650 3300
+Wire Wire Line
+	4200 3300 4200 3200
+Wire Wire Line
+	4200 2900 4200 2750
+Connection ~ 4200 2750
+Wire Wire Line
+	4200 2750 5050 2750
+Text HLabel 4850 3950 0    50   BiDi ~ 0
+SDA_1
+Text HLabel 4850 4050 0    50   Output ~ 0
+SCL_1
+Wire Wire Line
+	4850 3950 5050 3950
+Wire Wire Line
+	4850 4050 5050 4050
 $EndSCHEMATC
