File: robot/Object Detection.sch (KiCad schematic (older format))
At the start: 1 part

Commit message: DRC check fixes and small changes
Parts:
- gave numbers to parts that had none: 1
Changed lines of the file:
@@
 $EndDescr
 $Comp
-L Custom:CJVL53L0XV2 U?
+L Custom:CJVL53L0XV2 U4
 U 1 1 5D636DB5
 P 5750 4000
-F 0 "U?" H 5750 4565 50  0000 C CNN
+F 0 "U4" H 5750 4565 50  0000 C CNN
 F 1 "CJVL53L0XV2" H 5750 4474 50  0000 C CNN
 F 2 "" H 5750 4200 50  0001 C CNN
