File: robot/UI.sch (KiCad schematic (older format))
At the start: 11 parts

Commit message: DRC check fixes and small changes
Parts:
- gave numbers to parts that had none: 11
Other:
- moved on the sheet: D4, R16
Changed lines of the file:
@@
 $Descr A4 11693 8268
 encoding utf-8
-Sheet 8 8
+Sheet 7 8
 Title "User Interface"
 Date "2019-08-30"
@@
 $EndDescr
 $Comp
-L Device:LED D?
+L Device:LED D3
 U 1 1 5D6EDE25
 P 8150 4050
-F 0 "D?" V 8189 3933 50  0000 R CNN
+F 0 "D3" V 8189 3933 50  0000 R CNN
 F 1 "BLUE" V 8098 3933 50  0000 R CNN
 F 2 "" H 8150 4050 50  0001 C CNN
@@
 $EndComp
 $Comp
-L Device:R R?
+L Device:R R15
 U 1 1 5D6EE4EA
 P 8150 3500
-F 0 "R?" H 8080 3454 50  0000 R CNN
+F 0 "R15" H 8080 3454 50  0000 R CNN
 F 1 "150" H 8080 3545 50  0000 R CNN
 F 2 "" V 8080 3500 50  0001 C CNN
@@
 $EndComp
 $Comp
-L Custom:SSD1306 U?
+L Custom:SSD1306 U9
 U 1 1 5D6EEDF2
 P 5550 2850
-F 0 "U?" H 5450 2950 50  0000 L CNN
+F 0 "U9" H 5450 2950 50  0000 L CNN
 F 1 "SSD1306" H 5350 2850 50  0000 L CNN
 F 2 "" H 5550 2850 50  0001 C CNN
@@
 OLED 128x32
 $Comp
-L Device:C C?
+L Device:C C14
 U 1 1 5D6F2625
 P 4500 2950
-F 0 "C?" V 4450 2850 50  0000 C CNN
+F 0 "C14" V 4450 2850 50  0000 C CNN
 F 1 "1µ" V 4550 3050 50  0000 C CNN
 F 2 "" H 4538 2800 50  0001 C CNN
@@
 $EndComp
 $Comp
-L Device:C C?
+L Device:C C15
 U 1 1 5D6F2A4C
 P 4500 3250
-F 0 "C?" V 4450 3150 50  0000 C CNN
+F 0 "C15" V 4450 3150 50  0000 C CNN
 F 1 "1µ" V 4550 3350 50  0000 C CNN
 F 2 "" H 4538 3100 50  0001 C CNN
@@
 $EndComp
 $Comp
-L Device:C C?
+L Device:C C16
 U 1 1 5D6F3108
 P 4500 3550
-F 0 "C?" V 4450 3450 50  0000 C CNN
+F 0 "C16" V 4450 3450 50  0000 C CNN
 F 1 "1µ" V 4550 3650 50  0000 C CNN
 F 2 "" H 4538 3400 50  0001 C CNN
@@
 $EndComp
 $Comp
-L Device:C C?
+L Device:C C17
 U 1 1 5D6F3CE1
 P 4500 4750
-F 0 "C?" V 4450 4650 50  0000 C CNN
+F 0 "C17" V 4450 4650 50  0000 C CNN
 F 1 "4.7µ" V 4550 4900 50  0000 C CNN
 F 2 "" H 4538 4600 50  0001 C CNN
@@
 $EndComp
 $Comp
-L Device:C C?
+L Device:C C18
 U 1 1 5D6F35D1
 P 4500 5000
-F 0 "C?" V 4550 5100 50  0000 C CNN
+F 0 "C18" V 4550 5100 50  0000 C CNN
 F 1 "4.7µ" V 4450 4850 50  0000 C CNN
 F 2 "" H 4538 4850 50  0001 C CNN
@@
 $EndComp
 $Comp
-L Device:R R?
+L Device:R R17
 U 1 1 5D6F69C8
 P 4500 4550
-F 0 "R?" V 4550 4700 50  0000 C CNN
+F 0 "R17" V 4550 4700 50  0000 C CNN
 F 1 "330k" V 4450 4350 50  0000 C CNN
 F 2 "" V 4430 4550 50  0001 C CNN
@@
 	4050 3850 4050 4550
 $Comp
-L power:+3V3 #PWR?
+L power:+3V3 #PWR015
 U 1 1 5D6FA4C9
 P 3750 3900
-F 0 "#PWR?" H 3750 3750 50  0001 C CNN
+F 0 "#PWR015" H 3750 3750 50  0001 C CNN
 F 1 "+3V3" H 3765 4073 50  0000 C CNN
 F 2 "" H 3750 3900 50  0001 C CNN
@@
 	3750 4000 4800 4000
 $Comp
-L power:GND #PWR?
+L power:GND #PWR018
 U 1 1 5D6FB5BB
 P 4050 5200
-F 0 "#PWR?" H 4050 4950 50  0001 C CNN
+F 0 "#PWR018" H 4050 4950 50  0001 C CNN
 F 1 "GND" H 4055 5027 50  0000 C CNN
 F 2 "" H 4050 5200 50  0001 C CNN
@@
 	4800 4000 5050 4000
 $Comp
-L power:GND #PWR?
+L power:GND #PWR016
 U 1 1 5D6FEF4B
 P 8150 4400
-F 0 "#PWR?" H 8150 4150 50  0001 C CNN
+F 0 "#PWR016" H 8150 4150 50  0001 C CNN
 F 1 "GND" H 8155 4227 50  0000 C CNN
 F 2 "" H 8150 4400 50  0001 C CNN
@@
 Status LEDS
 $Comp
-L Device:LED D?
+L Device:LED D4
 U 1 1 5D760843
-P 8900 4050
-F 0 "D?" V 8939 3932 50  0000 R CNN
-F 1 "GREEN" V 8848 3932 50  0000 R CNN
-F 2 "" H 8900 4050 50  0001 C CNN
-F 3 "~" H 8900 4050 50  0001 C CNN
-	1    8900 4050
-	0    -1   -1   0
-$EndComp
-$Comp
-L Device:R R?
+P 9150 4050
+F 0 "D4" V 9189 3932 50  0000 R CNN
+F 1 "GREEN" V 9098 3932 50  0000 R CNN
+F 2 "" H 9150 4050 50  0001 C CNN
+F 3 "~" H 9150 4050 50  0001 C CNN
+	1    9150 4050
+	0    -1   -1   0
+$EndComp
+$Comp
+L Device:R R16
 U 1 1 5D76084D
-P 8900 3500
-F 0 "R?" H 8830 3454 50  0000 R CNN
-F 1 "150" H 8830 3545 50  0000 R CNN
-F 2 "" V 8830 3500 50  0001 C CNN
-F 3 "~" H 8900 3500 50  0001 C CNN
-	1    8900 3500
+P 9150 3500
+F 0 "R16" H 9080 3454 50  0000 R CNN
+F 1 "150" H 9080 3545 50  0000 R CNN
+F 2 "" V 9080 3500 50  0001 C CNN
+F 3 "~" H 9150 3500 50  0001 C CNN
+	1    9150 3500
 	-1   0    0    1
 $EndComp
 $Comp
-L power:GND #PWR?
+L power:GND #PWR017
 U 1 1 5D760857
-P 8900 4400
-F 0 "#PWR?" H 8900 4150 50  0001 C CNN
-F 1 "GND" H 8905 4227 50  0000 C CNN
-F 2 "" H 8900 4400 50  0001 C CNN
-F 3 "" H 8900 4400 50  0001 C CNN
-	1    8900 4400
-	1    0    0    -1
-$EndComp
-Wire Wire Line
-	8900 3650 8900 3900
-Wire Wire Line
-	8900 4200 8900 4400
-Wire Wire Line
-	8900 3350 8900 3150
-Wire Wire Line
-	8900 3150 8850 3150
-Text HLabel 8850 3150 0    50   Input ~ 0
+P 9150 4400
+F 0 "#PWR017" H 9150 4150 50  0001 C CNN
+F 1 "GND" H 9155 4227 50  0000 C CNN
+F 2 "" H 9150 4400 50  0001 C CNN
+F 3 "" H 9150 4400 50  0001 C CNN
+	1    9150 4400
+	1    0    0    -1
+$EndComp
+Wire Wire Line
+	9150 3650 9150 3900
+Wire Wire Line
+	9150 4200 9150 4400
+Wire Wire Line
+	9150 3350 9150 3150
+Wire Wire Line
+	9150 3150 9100 3150
+Text HLabel 9100 3150 0    50   Input ~ 0
 STATUS_LED_GRN
 $EndSCHEMATC

Commit message: Testpoints, switch, small changes
Changed lines of the file:
@@
 U 1 1 5D6F2625
 P 4500 2950
-F 0 "C14" V 4450 2850 50  0000 C CNN
+F 0 "C14" V 4450 2800 50  0000 C CNN
 F 1 "1µ" V 4550 3050 50  0000 C CNN
 F 2 "" H 4538 2800 50  0001 C CNN
@@
 U 1 1 5D6F2A4C
 P 4500 3250
-F 0 "C15" V 4450 3150 50  0000 C CNN
+F 0 "C15" V 4450 3100 50  0000 C CNN
 F 1 "1µ" V 4550 3350 50  0000 C CNN
 F 2 "" H 4538 3100 50  0001 C CNN
@@
 U 1 1 5D6F3108
 P 4500 3550
-F 0 "C16" V 4450 3450 50  0000 C CNN
+F 0 "C16" V 4450 3400 50  0000 C CNN
 F 1 "1µ" V 4550 3650 50  0000 C CNN
 F 2 "" H 4538 3400 50  0001 C CNN
@@
 U 1 1 5D6F3CE1
 P 4500 4750
-F 0 "C17" V 4450 4650 50  0000 C CNN
+F 0 "C17" V 4450 4600 50  0000 C CNN
 F 1 "4.7µ" V 4550 4900 50  0000 C CNN
 F 2 "" H 4538 4600 50  0001 C CNN
@@
 U 1 1 5D6F35D1
 P 4500 5000
-F 0 "C18" V 4550 5100 50  0000 C CNN
+F 0 "C18" V 4550 5150 50  0000 C CNN
 F 1 "4.7µ" V 4450 4850 50  0000 C CNN
 F 2 "" H 4538 4850 50  0001 C CNN
@@
 U 1 1 5D6F69C8
 P 4500 4550
-F 0 "R17" V 4550 4700 50  0000 C CNN
+F 0 "R17" V 4550 4750 50  0000 C CNN
 F 1 "330k" V 4450 4350 50  0000 C CNN
 F 2 "" V 4430 4550 50  0001 C CNN
@@
 	4050 3850 4050 4550
 $Comp
-L power:+3V3 #PWR015
+L power:+3V3 #PWR042
 U 1 1 5D6FA4C9
 P 3750 3900
-F 0 "#PWR015" H 3750 3750 50  0001 C CNN
+F 0 "#PWR042" H 3750 3750 50  0001 C CNN
 F 1 "+3V3" H 3765 4073 50  0000 C CNN
 F 2 "" H 3750 3900 50  0001 C CNN
@@
 	3750 4000 4800 4000
 $Comp
-L power:GND #PWR018
+L power:GND #PWR045
 U 1 1 5D6FB5BB
 P 4050 5200
-F 0 "#PWR018" H 4050 4950 50  0001 C CNN
+F 0 "#PWR045" H 4050 4950 50  0001 C CNN
 F 1 "GND" H 4055 5027 50  0000 C CNN
 F 2 "" H 4050 5200 50  0001 C CNN
@@
 	4800 4000 5050 4000
 $Comp
-L power:GND #PWR016
+L power:GND #PWR043
 U 1 1 5D6FEF4B
 P 8150 4400
-F 0 "#PWR016" H 8150 4150 50  0001 C CNN
+F 0 "#PWR043" H 8150 4150 50  0001 C CNN
 F 1 "GND" H 8155 4227 50  0000 C CNN
 F 2 "" H 8150 4400 50  0001 C CNN
@@
 $EndComp
 $Comp
-L power:GND #PWR017
+L power:GND #PWR044
 U 1 1 5D760857
 P 9150 4400
-F 0 "#PWR017" H 9150 4150 50  0001 C CNN
+F 0 "#PWR044" H 9150 4150 50  0001 C CNN
 F 1 "GND" H 9155 4227 50  0000 C CNN
 F 2 "" H 9150 4400 50  0001 C CNN
