File: robot/Front/Front.sch (KiCad schematic (older format))
At the start: 20 parts, among them Q1 BC849, Q2 BC849, SW2 SW_Push, U1 CH340G, U10 ESP32-WROOM-32, U2 CJVL53L0XV2, Y1 Crystal_GND24

Commit message: Cleanup, start PDB Front
Parts:
- removed C4, C5: 22p, symbol Device:C
- removed Y1: Crystal_GND24, symbol Device:Crystal_GND24
- added C6: 10µ, Capacitors_SMD:C_1206_HandSoldering, symbol Device:C
- added H1: VBUS, Custom:Mounting_Pad_Power, symbol Custom:MountingPad
- added H10: M1B2, Custom:Mounting_Pad_Signal, symbol Custom:MountingPad
- added H11: BAT_MON, Custom:Mounting_Pad_Signal, symbol Custom:MountingPad
- added H12: ED1, Custom:Mounting_Pad_Signal, symbol Custom:MountingPad
- added H13: ED2, Custom:Mounting_Pad_Signal, symbol Custom:MountingPad
- added H14: OSDA, Custom:Mounting_Pad_Signal, symbol Custom:MountingPad
- added H15: OSCL, Custom:Mounting_Pad_Signal, symbol Custom:MountingPad
- added H16: ORST, Custom:Mounting_Pad_Signal, symbol Custom:MountingPad
- added H17: VBAT_SWITCH, Custom:Mounting_Pad_Power, symbol Custom:MountingPad
- added H18, H19, H21, H22: GND, Custom:Mounting_Pad_Power, symbol Custom:MountingPad
- added H2: M_~SLP, Custom:Mounting_Pad_Signal, symbol Custom:MountingPad
- added H20, H23: 3V3, Custom:Mounting_Pad_Power, symbol Custom:MountingPad
- added H3: M2B2, Custom:Mounting_Pad_Signal, symbol Custom:MountingPad
- added H4: M2B1, Custom:Mounting_Pad_Signal, symbol Custom:MountingPad
- added H5: M2A2, Custom:Mounting_Pad_Signal, symbol Custom:MountingPad
- added H6: M2A1, Custom:Mounting_Pad_Signal, symbol Custom:MountingPad
- added H7: M1A1, Custom:Mounting_Pad_Signal, symbol Custom:MountingPad
- added H8: M1A2, Custom:Mounting_Pad_Signal, symbol Custom:MountingPad
- added H9: M1B1, Custom:Mounting_Pad_Signal, symbol Custom:MountingPad
- added J1: USB_B_Micro, Connectors_USB:USB_Micro-B_Molex_47346-0001, symbol Connector:USB_B_Micro
- added U3: LD1117S33CTR, digikey-footprints:SOT-223, symbol dk_PMIC-Voltage-Regulators-Linear:LD1117S33CTR
- C1, C19, C2, C3: footprint (none) -> Capacitors_SMD:C_1206_HandSoldering
- D1, D2: footprint (none) -> LED_SMD:LED_0805_2012Metric_Pad1.15x1.40mm_HandSolder
- R1, R18, R2, R3, R4: footprint (none) -> Resistors_SMD:R_1206_HandSoldering
- SW2: footprint (none) -> Buttons_Switches_THT:SW_PUSH_SMALL
- U1: value CH340G -> CH340C
- U2: footprint (none) -> Custom:CJVL53L0XV2
Connections:
- net labels added: OLED_SCL, OLED_SDA
- net labels removed: SCL_1, SDA_1, USB_D+, USB_D-
- wire segments 107 -> 134
- no-connect marks 13 -> 16
Other:
- note added: "PADS BOTTOM"
- note added: "PADS TOP"
- note added: "VDO"
- moved on the sheet: C3, D1, D2, Q1, Q2, R1, R2, R4

Commit message: Front PCB
Parts:
- removed C19: 1µ, Capacitors_SMD:C_1206_HandSoldering, symbol Device:C
- C1, C2, C3, C6: footprint Capacitors_SMD:C_1206_HandSoldering -> Capacitors_SMD:C_1206
- R1, R18, R2, R3, R4: footprint Resistors_SMD:R_1206_HandSoldering -> Resistors_SMD:R_1206
- SW2: footprint Buttons_Switches_THT:SW_PUSH_SMALL -> Button_Switch_SMD:Panasonic_EVQPUJ_EVQPUA
- U2: footprint Custom:CJVL53L0XV2 -> Custom:CJVL53L0XV2_NoMountHoles; symbol Custom:CJVL53L0XV2 -> Custom:CJVL53L0XV2_NoMountingHoles
- U3: footprint digikey-footprints:SOT-223 -> Package_TO_SOT_SMD:SOT-223
Other:
- moved on the sheet: R18, SW2
Changed lines of the file:
@@
 	9850 1750 10050 1750
 Wire Wire Line
-	7000 1450 7250 1450
+	7750 1450 8000 1450
 Wire Wire Line
 	9850 1450 10050 1450
-$Comp
-L Device:C C19
-U 1 1 5D72A799
-P 7800 1750
-F 0 "C19" H 7915 1796 50  0000 L CNN
-F 1 "1µ" H 7915 1705 50  0000 L CNN
-F 2 "Capacitors_SMD:C_1206_HandSoldering" H 7838 1600 50  0001 C CNN
-F 3 "~" H 7800 1750 50  0001 C CNN
-	1    7800 1750
-	1    0    0    -1
-$EndComp
 $Comp
 L Switch:SW_Push SW2
 U 1 1 5D62C889
-P 7250 1800
-F 0 "SW2" V 7350 1650 50  0000 C CNN
-F 1 "SW_Push" V 7200 1550 50  0000 C CNN
-F 2 "Buttons_Switches_THT:SW_PUSH_SMALL" H 7250 2000 50  0001 C CNN
-F 3 "~" H 7250 2000 50  0001 C CNN
-	1    7250 1800
+P 8000 1800
+F 0 "SW2" V 8100 1650 50  0000 C CNN
+F 1 "SW_Push" V 7950 1550 50  0000 C CNN
+F 2 "Button_Switch_SMD:Panasonic_EVQPUJ_EVQPUA" H 8000 2000 50  0001 C CNN
+F 3 "~" H 8000 2000 50  0001 C CNN
+	1    8000 1800
 	0    -1   -1   0
 $EndComp
@@
 L Device:R R18
 U 1 1 5D62DCB0
-P 7250 1150
-F 0 "R18" H 7320 1196 50  0000 L CNN
-F 1 "10k" H 7320 1105 50  0000 L CNN
-F 2 "Resistors_SMD:R_1206_HandSoldering" V 7180 1150 50  0001 C CNN
-F 3 "~" H 7250 1150 50  0001 C CNN
-	1    7250 1150
+P 8000 1150
+F 0 "R18" H 8070 1196 50  0000 L CNN
+F 1 "10k" H 8070 1105 50  0000 L CNN
+F 2 "Resistors_SMD:R_1206" V 7930 1150 50  0001 C CNN
+F 3 "~" H 8000 1150 50  0001 C CNN
+	1    8000 1150
 	1    0    0    -1
 $EndComp
@@
 L power:+3V3 #PWR046
 U 1 1 5D62E308
-P 7250 900
-F 0 "#PWR046" H 7250 750 50  0001 C CNN
-F 1 "+3V3" H 7265 1073 50  0000 C CNN
-F 2 "" H 7250 900 50  0001 C CNN
-F 3 "" H 7250 900 50  0001 C CNN
-	1    7250 900
+P 8000 900
+F 0 "#PWR046" H 8000 750 50  0001 C CNN
+F 1 "+3V3" H 8015 1073 50  0000 C CNN
+F 2 "" H 8000 900 50  0001 C CNN
+F 3 "" H 8000 900 50  0001 C CNN
+	1    8000 900
 	1    0    0    -1
 $EndComp
@@
 L power:GND #PWR049
 U 1 1 5D62E7C3
-P 7250 2100
-F 0 "#PWR049" H 7250 1850 50  0001 C CNN
-F 1 "GND" H 7255 1927 50  0000 C CNN
-F 2 "" H 7250 2100 50  0001 C CNN
-F 3 "" H 7250 2100 50  0001 C CNN
-	1    7250 2100
-	1    0    0    -1
-$EndComp
-$Comp
-L power:GND #PWR048
-U 1 1 5D62EDF6
-P 7800 2000
-F 0 "#PWR048" H 7800 1750 50  0001 C CNN
-F 1 "GND" H 7805 1827 50  0000 C CNN
-F 2 "" H 7800 2000 50  0001 C CNN
-F 3 "" H 7800 2000 50  0001 C CNN
-	1    7800 2000
-	1    0    0    -1
-$EndComp
-Wire Wire Line
-	7250 900  7250 1000
-Wire Wire Line
-	7250 1300 7250 1450
-Connection ~ 7250 1450
-Wire Wire Line
-	7250 1450 7800 1450
-Wire Wire Line
-	7250 1600 7250 1450
-Wire Wire Line
-	7250 2100 7250 2000
-Wire Wire Line
-	7800 2000 7800 1900
-Wire Wire Line
-	7800 1600 7800 1450
-Connection ~ 7800 1450
-Wire Wire Line
-	7800 1450 8650 1450
+P 8000 2100
+F 0 "#PWR049" H 8000 1850 50  0001 C CNN
+F 1 "GND" H 8005 1927 50  0000 C CNN
+F 2 "" H 8000 2100 50  0001 C CNN
+F 3 "" H 8000 2100 50  0001 C CNN
+	1    8000 2100
+	1    0    0    -1
+$EndComp
+Wire Wire Line
+	8000 900  8000 1000
+Wire Wire Line
+	8000 1300 8000 1450
+Connection ~ 8000 1450
+Wire Wire Line
+	8000 1600 8000 1450
+Wire Wire Line
+	8000 2100 8000 2000
 Wire Wire Line
 	9850 2050 10050 2050
@@
 F 0 "C1" H 2365 1846 50  0000 L CNN
 F 1 "100n" H 2365 1755 50  0000 L CNN
-F 2 "Capacitors_SMD:C_1206_HandSoldering" H 2288 1650 50  0001 C CNN
+F 2 "Capacitors_SMD:C_1206" H 2288 1650 50  0001 C CNN
 F 3 "~" H 2250 1800 50  0001 C CNN
 	1    2250 1800
@@
 F 0 "C3" H 4565 1896 50  0000 L CNN
 F 1 "100n" H 4565 1805 50  0000 L CNN
-F 2 "Capacitors_SMD:C_1206_HandSoldering" H 4488 1700 50  0001 C CNN
+F 2 "Capacitors_SMD:C_1206" H 4488 1700 50  0001 C CNN
 F 3 "~" H 4450 1850 50  0001 C CNN
 	1    4450 1850
@@
 F 0 "C2" H 4165 1896 50  0000 L CNN
 F 1 "10µ" H 4165 1805 50  0000 L CNN
-F 2 "Capacitors_SMD:C_1206_HandSoldering" H 4088 1700 50  0001 C CNN
+F 2 "Capacitors_SMD:C_1206" H 4088 1700 50  0001 C CNN
 F 3 "~" H 4050 1850 50  0001 C CNN
 	1    4050 1850
@@
 F 0 "R1" V 4250 2650 50  0000 C CNN
 F 1 "10k" V 4050 2650 50  0000 C CNN
-F 2 "Resistors_SMD:R_1206_HandSoldering" V 4080 2650 50  0001 C CNN
+F 2 "Resistors_SMD:R_1206" V 4080 2650 50  0001 C CNN
 F 3 "~" H 4150 2650 50  0001 C CNN
 	1    4150 2650
@@
 F 0 "R2" V 4250 3350 50  0000 C CNN
 F 1 "10k" V 4034 3350 50  0000 C CNN
-F 2 "Resistors_SMD:R_1206_HandSoldering" V 4080 3350 50  0001 C CNN
+F 2 "Resistors_SMD:R_1206" V 4080 3350 50  0001 C CNN
 F 3 "~" H 4150 3350 50  0001 C CNN
 	1    4150 3350
@@
 F 0 "R3" H 9630 5254 50  0000 R CNN
 F 1 "150" H 9630 5345 50  0000 R CNN
-F 2 "Resistors_SMD:R_1206_HandSoldering" V 9630 5300 50  0001 C CNN
+F 2 "Resistors_SMD:R_1206" V 9630 5300 50  0001 C CNN
 F 3 "~" H 9700 5300 50  0001 C CNN
 	1    9700 5300
@@
 F 0 "R4" H 10630 5254 50  0000 R CNN
 F 1 "150" H 10630 5345 50  0000 R CNN
-F 2 "Resistors_SMD:R_1206_HandSoldering" V 10630 5300 50  0001 C CNN
+F 2 "Resistors_SMD:R_1206" V 10630 5300 50  0001 C CNN
 F 3 "~" H 10700 5300 50  0001 C CNN
 	1    10700 5300
@@
 	10700 5000 10650 5000
 $Comp
-L Custom:CJVL53L0XV2 U2
+L Custom:CJVL53L0XV2_NoMountingHoles U2
 U 1 1 5D72A7B2
 P 7800 5000
 F 0 "U2" H 7800 5565 50  0000 C CNN
 F 1 "CJVL53L0XV2" H 7800 5474 50  0000 C CNN
-F 2 "Custom:CJVL53L0XV2" H 7800 5200 50  0001 C CNN
+F 2 "Custom:CJVL53L0XV2_NoMountHoles" H 7800 5200 50  0001 C CNN
 F 3 "" H 7800 5200 50  0001 C CNN
 	1    7800 5000
@@
 Text Label 10650 5000 2    50   ~ 0
 STATUS_LED_GRN
-Text Label 7000 1450 2    50   ~ 0
+Text Label 7750 1450 2    50   ~ 0
 ~RST
 Text Label 10050 1450 0    50   ~ 0
@@
 F 0 "C6" H 2765 6096 50  0000 L CNN
 F 1 "10µ" H 2765 6005 50  0000 L CNN
-F 2 "Capacitors_SMD:C_1206_HandSoldering" H 2688 5900 50  0001 C CNN
+F 2 "Capacitors_SMD:C_1206" H 2688 5900 50  0001 C CNN
 F 3 "~" H 2650 6050 50  0001 C CNN
 	1    2650 6050
@@
 F 0 "U3" H 2000 6137 60  0000 C CNN
 F 1 "LD1117S33CTR" H 2000 6031 60  0000 C CNN
-F 2 "digikey-footprints:SOT-223" H 2150 6050 60  0001 L CNN
+F 2 "Package_TO_SOT_SMD:SOT-223" H 2150 6050 60  0001 L CNN
 F 3 "http://www.st.com/content/ccc/resource/technical/document/datasheet/99/3b/7d/91/91/51/4b/be/CD00000544.pdf/files/CD00000544.pdf/jcr:content/translations/en.CD00000544.pdf" H 2150 6150 60  0001 L CNN
 F 4 "497-1241-1-ND" H 2150 6250 60  0001 L CNN "Digi-Key_PN"
@@
 NoConn ~ 2350 2850
 NoConn ~ 2350 3050
+Wire Wire Line
+	8000 1450 8650 1450
 $EndSCHEMATC

Commit message: Front Routing
Parts:
- added H24: 3V3, Custom:Mounting_Pad_Power, symbol Custom:MountingPad
Connections:
- net +3V3: now also C2.1, C3.1, U1.16 (VCC), H24.1 (Pin)
- net VBUS: no longer C2.1, C3.1, U1.16 (VCC)
- net D+: now reaches J1.3 (D+), U1.5 (UD+)
- net D-: now reaches J1.2 (D-), U1.6 (UD-)
Other:
- moved on the sheet: H18, H19
Changed lines of the file:
@@
-	1    0    0    -1
-$EndComp
-$Comp
-L power:VBUS #PWR?
-U 1 1 5D7276F4
-P 2750 1350
-AR Path="/5D17B31F/5D7276F4" Ref="#PWR?"  Part="1"
-AR Path="/5D179377/5D7276F4" Ref="#PWR?"  Part="1"
-AR Path="/5D7276F4" Ref="#PWR01"  Part="1"
-F 0 "#PWR01" H 2750 1200 50  0001 C CNN
-F 1 "VBUS" H 2765 1523 50  0000 C CNN
-F 2 "" H 2750 1350 50  0001 C CNN
-F 3 "" H 2750 1350 50  0001 C CNN
-	1    2750 1350
 	1    0    0    -1
 $EndComp
@@
 L Custom:MountingPad H18
 U 1 1 5D850133
-P 4600 5500
-F 0 "H18" H 4550 5550 50  0000 R CNN
-F 1 "GND" H 4550 5450 50  0000 R CNN
-F 2 "Custom:Mounting_Pad_Power" H 4600 5650 50  0001 C CNN
-F 3 "" H 4600 5650 50  0001 C CNN
-	1    4600 5500
+P 4500 5500
+F 0 "H18" H 4450 5550 50  0000 R CNN
+F 1 "GND" H 4450 5450 50  0000 R CNN
+F 2 "Custom:Mounting_Pad_Power" H 4500 5650 50  0001 C CNN
+F 3 "" H 4500 5650 50  0001 C CNN
+	1    4500 5500
 	1    0    0    -1
 $EndComp
@@
 L Custom:MountingPad H19
 U 1 1 5D850139
-P 4900 5500
-F 0 "H19" H 5050 5550 50  0000 R CNN
-F 1 "GND" H 5100 5450 50  0000 R CNN
-F 2 "Custom:Mounting_Pad_Power" H 4900 5650 50  0001 C CNN
-F 3 "" H 4900 5650 50  0001 C CNN
-	1    4900 5500
+P 5000 5500
+F 0 "H19" H 5150 5550 50  0000 R CNN
+F 1 "GND" H 5200 5450 50  0000 R CNN
+F 2 "Custom:Mounting_Pad_Power" H 5000 5650 50  0001 C CNN
+F 3 "" H 5000 5650 50  0001 C CNN
+	1    5000 5500
 	1    0    0    -1
 $EndComp
@@
 L power:GND #PWR018
 U 1 1 5D85013F
-P 4600 5800
-F 0 "#PWR018" H 4600 5550 50  0001 C CNN
-F 1 "GND" H 4605 5627 50  0000 C CNN
-F 2 "" H 4600 5800 50  0001 C CNN
-F 3 "" H 4600 5800 50  0001 C CNN
-	1    4600 5800
+P 4500 5800
+F 0 "#PWR018" H 4500 5550 50  0001 C CNN
+F 1 "GND" H 4505 5627 50  0000 C CNN
+F 2 "" H 4500 5800 50  0001 C CNN
+F 3 "" H 4500 5800 50  0001 C CNN
+	1    4500 5800
 	1    0    0    -1
 $EndComp
@@
 L power:GND #PWR019
 U 1 1 5D850145
-P 4900 5800
-F 0 "#PWR019" H 4900 5550 50  0001 C CNN
-F 1 "GND" H 4905 5627 50  0000 C CNN
-F 2 "" H 4900 5800 50  0001 C CNN
-F 3 "" H 4900 5800 50  0001 C CNN
-	1    4900 5800
-	1    0    0    -1
-$EndComp
-Text Notes 4550 5200 0    50   ~ 0
+P 5000 5800
+F 0 "#PWR019" H 5000 5550 50  0001 C CNN
+F 1 "GND" H 5005 5627 50  0000 C CNN
+F 2 "" H 5000 5800 50  0001 C CNN
+F 3 "" H 5000 5800 50  0001 C CNN
+	1    5000 5800
+	1    0    0    -1
+$EndComp
+Text Notes 4600 4800 0    50   ~ 0
 PADS TOP
 Wire Wire Line
@@
 Wire Wire Line
 	8000 1450 8650 1450
+$Comp
+L Custom:MountingPad H24
+U 1 1 5D7A096E
+P 4750 5500
+F 0 "H24" H 4700 5450 50  0000 R CNN
+F 1 "3V3" H 4700 5550 50  0000 R CNN
+F 2 "Custom:Mounting_Pad_Power" H 4750 5650 50  0001 C CNN
+F 3 "" H 4750 5650 50  0001 C CNN
+	1    4750 5500
+	-1   0    0    1
+$EndComp
+$Comp
+L power:+3V3 #PWR04
+U 1 1 5D7A0978
+P 4750 5100
+F 0 "#PWR04" H 4750 4950 50  0001 C CNN
+F 1 "+3V3" H 4765 5273 50  0000 C CNN
+F 2 "" H 4750 5100 50  0001 C CNN
+F 3 "" H 4750 5100 50  0001 C CNN
+	1    4750 5100
+	1    0    0    -1
+$EndComp
+Wire Wire Line
+	4750 5100 4750 5200
+$Comp
+L power:+3V3 #PWR0101
+U 1 1 5D7D9324
+P 2750 1350
+F 0 "#PWR0101" H 2750 1200 50  0001 C CNN
+F 1 "+3V3" H 2765 1523 50  0000 C CNN
+F 2 "" H 2750 1350 50  0001 C CNN
+F 3 "" H 2750 1350 50  0001 C CNN
+	1    2750 1350
+	1    0    0    -1
+$EndComp
+Text Label 1500 2100 0    50   ~ 0
+D+
+Text Label 1500 2200 0    50   ~ 0
+D-
 $EndSCHEMATC

Commit message: Renumber and more Bottom
Parts:
- H10: value M1B2 -> M2B2
- H17: value VBAT_SWITCH -> VBS
- H3: value M2B2 -> M1B2
- H4: value M2B1 -> M1B1
- H5: value M2A2 -> M1A2
- H6: value M2A1 -> M1A1
- H7: value M1A1 -> M2A1
- H8: value M1A2 -> M2A2
- H9: value M1B1 -> M2B1
Connections:
- net M1_AOUT1: now also H6.1 (Pin), U10.19 (SCS/CMD); no longer H7.1 (Pin), U10.20 (SCK/CLK)
- net M1_AOUT2: now also H5.1 (Pin), U10.18 (SWP/SD3); no longer H8.1 (Pin), U10.21 (SDO/SD0)
- net M1_BOUT1: now also H4.1 (Pin), U10.17 (SHD/SD2); no longer H9.1 (Pin), U10.22 (SDI/SD1)
- net M1_BOUT2: now also H3.1 (Pin), U10.16 (IO13); no longer H10.1 (Pin), U10.23 (IO15)
- net M2_AOUT1: now also H7.1 (Pin), U10.20 (SCK/CLK); no longer H6.1 (Pin), U10.19 (SCS/CMD)
- net M2_AOUT2: now also H8.1 (Pin), U10.21 (SDO/SD0); no longer H5.1 (Pin), U10.18 (SWP/SD3)
- net M2_BOUT1: now also H9.1 (Pin), U10.22 (SDI/SD1); no longer H4.1 (Pin), U10.17 (SHD/SD2)
- net M2_BOUT2: now also H10.1 (Pin), U10.23 (IO15); no longer H3.1 (Pin), U10.16 (IO13)
Changed lines of the file:
@@
 OD_SHUT
 Text Label 8450 2650 2    50   ~ 0
+M2_AOUT2
+Text Label 8450 2750 2    50   ~ 0
+M2_BOUT1
+Text Label 8450 2850 2    50   ~ 0
+M1_BOUT1
+Text Label 8450 2950 2    50   ~ 0
 M1_AOUT2
-Text Label 8450 2750 2    50   ~ 0
-M1_BOUT1
-Text Label 8450 2850 2    50   ~ 0
-M2_BOUT1
-Text Label 8450 2950 2    50   ~ 0
-M2_AOUT2
 Text Label 8450 3050 2    50   ~ 0
+M2_AOUT1
+Text Label 8450 3150 2    50   ~ 0
 M1_AOUT1
-Text Label 8450 3150 2    50   ~ 0
-M2_AOUT1
 Text Label 10050 3750 0    50   ~ 0
 ED_IN2
@@
 OLED_SDA
 Text Label 10050 2350 0    50   ~ 0
+M2_BOUT2
+Text Label 10050 2150 0    50   ~ 0
 M1_BOUT2
-Text Label 10050 2150 0    50   ~ 0
-M2_BOUT2
 Text Label 10050 1650 0    50   ~ 0
 M1_M2_~SLEEP
@@
 P 1350 5350
 F 0 "H17" H 1438 5288 50  0000 L CNN
-F 1 "VBAT_SWITCH" H 1438 5197 50  0000 L CNN
+F 1 "VBS" H 1438 5197 50  0000 L CNN
 F 2 "Custom:Mounting_Pad_Power" H 1350 5500 50  0001 C CNN
 F 3 "" H 1350 5500 50  0001 C CNN
@@
 P 6150 3350
 F 0 "H3" H 6350 3300 50  0000 R CNN
-F 1 "M2B2" H 6250 3500 50  0000 R CNN
+F 1 "M1B2" H 6250 3500 50  0000 R CNN
 F 2 "Custom:Mounting_Pad_Signal" H 6150 3500 50  0001 C CNN
 F 3 "" H 6150 3500 50  0001 C CNN
@@
 P 6400 3350
 F 0 "H4" H 6600 3300 50  0000 R CNN
-F 1 "M2B1" H 6500 3500 50  0000 R CNN
+F 1 "M1B1" H 6500 3500 50  0000 R CNN
 F 2 "Custom:Mounting_Pad_Signal" H 6400 3500 50  0001 C CNN
 F 3 "" H 6400 3500 50  0001 C CNN
@@
 P 6650 3350
 F 0 "H5" H 6850 3300 50  0000 R CNN
-F 1 "M2A2" H 6750 3500 50  0000 R CNN
+F 1 "M1A2" H 6750 3500 50  0000 R CNN
 F 2 "Custom:Mounting_Pad_Signal" H 6650 3500 50  0001 C CNN
 F 3 "" H 6650 3500 50  0001 C CNN
@@
 P 6900 3350
 F 0 "H6" H 7100 3300 50  0000 R CNN
-F 1 "M2A1" H 7000 3500 50  0000 R CNN
+F 1 "M1A1" H 7000 3500 50  0000 R CNN
 F 2 "Custom:Mounting_Pad_Signal" H 6900 3500 50  0001 C CNN
 F 3 "" H 6900 3500 50  0001 C CNN
@@
 P 7150 3350
 F 0 "H7" H 7350 3300 50  0000 R CNN
-F 1 "M1A1" H 7250 3500 50  0000 R CNN
+F 1 "M2A1" H 7250 3500 50  0000 R CNN
 F 2 "Custom:Mounting_Pad_Signal" H 7150 3500 50  0001 C CNN
 F 3 "" H 7150 3500 50  0001 C CNN
@@
 P 7400 3350
 F 0 "H8" H 7600 3300 50  0000 R CNN
-F 1 "M1A2" H 7500 3500 50  0000 R CNN
+F 1 "M2A2" H 7500 3500 50  0000 R CNN
 F 2 "Custom:Mounting_Pad_Signal" H 7400 3500 50  0001 C CNN
 F 3 "" H 7400 3500 50  0001 C CNN
@@
 P 7650 3350
 F 0 "H9" H 7850 3300 50  0000 R CNN
-F 1 "M1B1" H 7750 3500 50  0000 R CNN
+F 1 "M2B1" H 7750 3500 50  0000 R CNN
 F 2 "Custom:Mounting_Pad_Signal" H 7650 3500 50  0001 C CNN
 F 3 "" H 7650 3500 50  0001 C CNN
@@
 P 7900 3350
 F 0 "H10" H 8100 3300 50  0000 R CNN
-F 1 "M1B2" H 8000 3500 50  0000 R CNN
+F 1 "M2B2" H 8000 3500 50  0000 R CNN
 F 2 "Custom:Mounting_Pad_Signal" H 7900 3500 50  0001 C CNN
 F 3 "" H 7900 3500 50  0001 C CNN
@@
 $EndComp
 Text Label 6150 2950 1    50   ~ 0
+M1_BOUT2
+Text Label 6400 2950 1    50   ~ 0
+M1_BOUT1
+Text Label 6650 2950 1    50   ~ 0
+M1_AOUT2
+Text Label 6900 2950 1    50   ~ 0
+M1_AOUT1
+Text Label 7150 2950 1    50   ~ 0
+M2_AOUT1
+Text Label 7400 2950 1    50   ~ 0
+M2_AOUT2
+Text Label 7650 2950 1    50   ~ 0
+M2_BOUT1
+Text Label 7900 2950 1    50   ~ 0
 M2_BOUT2
-Text Label 6400 2950 1    50   ~ 0
-M2_BOUT1
-Text Label 6650 2950 1    50   ~ 0
-M2_AOUT2
-Text Label 6900 2950 1    50   ~ 0
-M2_AOUT1
-Text Label 7150 2950 1    50   ~ 0
-M1_AOUT1
-Text Label 7400 2950 1    50   ~ 0
-M1_AOUT2
-Text Label 7650 2950 1    50   ~ 0
-M1_BOUT1
-Text Label 7900 2950 1    50   ~ 0
-M1_BOUT2
 Wire Wire Line
 	6150 2950 6150 3050
