File: robot/Front/Front.sch (KiCad schematic (older format))
At the start: 41 parts, among them J1 USB_B_Micro, Q1 BC849, Q2 BC849, SW2 SW_Push, U1 CH340C, U10 ESP32-WROOM-32, U2 CJVL53L0XV2, U3 SPX3819M5-L-3-3

Commit message: Small changes, BOM, Gerbers
Parts:
- C1: LCSC (none) -> C282732
- C2: LCSC (none) -> C5674
- D1: LCSC (none) -> C84259
- D2: LCSC (none) -> C84260
- H11: value BAT_MON -> BTMN
- H2: value M_~SLP -> M~SLP
- J1: Farnell (none) -> 2782045; LCSC (none) -> C40942
- Q1, Q2: LCSC (none) -> C163753
- R1, R18, R2: LCSC (none) -> C38522
- R3, R4: LCSC (none) -> C25283
- SW2: Farnell (none) -> 2860922
- U1: LCSC (none) -> C84681
- U3: LCSC (none) -> C9055
Changed lines of the file:
@@
 F 2 "Button_Switch_SMD:Panasonic_EVQPUJ_EVQPUA" H 7700 2000 50  0001 C CNN
 F 3 "~" H 7700 2000 50  0001 C CNN
+F 4 "2860922" H 7700 1800 50  0001 C CNN "Farnell"
 	1    7700 1800
 	0    -1   -1   0
@@
 F 2 "Resistor_SMD:R_0805_2012Metric" V 7630 1150 50  0001 C CNN
 F 3 "~" H 7700 1150 50  0001 C CNN
+F 4 "C38522" H 7700 1150 50  0001 C CNN "LCSC"
 	1    7700 1150
 	1    0    0    -1
@@
 F 2 "Capacitor_SMD:C_0805_2012Metric" H 2288 1650 50  0001 C CNN
 F 3 "~" H 2250 1800 50  0001 C CNN
+F 4 "C282732" H 2250 1800 50  0001 C CNN "LCSC"
 	1    2250 1800
 	1    0    0    -1
@@
 F 2 "Capacitor_SMD:C_0805_2012Metric" H 4088 1700 50  0001 C CNN
 F 3 "~" H 4050 1850 50  0001 C CNN
+F 4 "C5674" H 4050 1850 50  0001 C CNN "LCSC"
 	1    4050 1850
 	1    0    0    -1
@@
 F 2 "Package_TO_SOT_SMD:SOT-23" H 4800 2575 50  0001 L CIN
 F 3 "http://www.infineon.com/dgdl/Infineon-BC847SERIES_BC848SERIES_BC849SERIES_BC850SERIES-DS-v01_01-en.pdf?fileId=db3a304314dca389011541d4630a1657" H 4600 2650 50  0001 L CNN
+F 4 "C163753" H 4600 2650 50  0001 C CNN "LCSC"
 	1    4600 2650
 	1    0    0    -1
@@
 F 2 "Package_TO_SOT_SMD:SOT-23" H 4800 3275 50  0001 L CIN
 F 3 "http://www.infineon.com/dgdl/Infineon-BC847SERIES_BC848SERIES_BC849SERIES_BC850SERIES-DS-v01_01-en.pdf?fileId=db3a304314dca389011541d4630a1657" H 4600 3350 50  0001 L CNN
+F 4 "C163753" H 4600 3350 50  0001 C CNN "LCSC"
 	1    4600 3350
 	1    0    0    1
@@
 F 2 "Resistor_SMD:R_0805_2012Metric" V 4080 2650 50  0001 C CNN
 F 3 "~" H 4150 2650 50  0001 C CNN
+F 4 "C38522" H 4150 2650 50  0001 C CNN "LCSC"
 	1    4150 2650
 	0    -1   -1   0
@@
 F 2 "Resistor_SMD:R_0805_2012Metric" V 4080 3350 50  0001 C CNN
 F 3 "~" H 4150 3350 50  0001 C CNN
+F 4 "C38522" H 4150 3350 50  0001 C CNN "LCSC"
 	1    4150 3350
 	0    1    1    0
@@
 F 2 "LED_SMD:LED_0805_2012Metric_Pad1.15x1.40mm_HandSolder" H 9700 5650 50  0001 C CNN
 F 3 "~" H 9700 5650 50  0001 C CNN
+F 4 "C84259" H 9700 5650 50  0001 C CNN "LCSC"
 	1    9700 5650
 	0    -1   -1   0
@@
 F 2 "Resistor_SMD:R_0805_2012Metric" V 9630 5300 50  0001 C CNN
 F 3 "~" H 9700 5300 50  0001 C CNN
+F 4 "C25283" H 9700 5300 50  0001 C CNN "LCSC"
 	1    9700 5300
 	-1   0    0    1
@@
 F 2 "LED_SMD:LED_0805_2012Metric_Pad1.15x1.40mm_HandSolder" H 10700 5650 50  0001 C CNN
 F 3 "~" H 10700 5650 50  0001 C CNN
+F 4 "C84260" H 10700 5650 50  0001 C CNN "LCSC"
 	1    10700 5650
 	0    -1   -1   0
@@
 F 2 "Resistor_SMD:R_0805_2012Metric" V 10630 5300 50  0001 C CNN
 F 3 "~" H 10700 5300 50  0001 C CNN
+F 4 "C25283" H 10700 5300 50  0001 C CNN "LCSC"
 	1    10700 5300
 	-1   0    0    1
@@
 F 2 "Connector_USB:USB_Micro-B_Molex_47346-0001" H 1250 2050 50  0001 C CNN
 F 3 "~" H 1250 2050 50  0001 C CNN
+F 4 "C40942" H 1100 2100 50  0001 C CNN "LCSC"
+F 5 "2782045" H 1100 2100 50  0001 C CNN "Farnell"
 	1    1100 2100
 	1    0    0    -1
@@
 P 5850 4300
 F 0 "H11" H 6050 4250 50  0000 R CNN
-F 1 "BAT_MON" H 6050 4450 50  0000 R CNN
+F 1 "BTMN" H 6050 4450 50  0000 R CNN
 F 2 "Custom:Mounting_Pad_Signal" H 5850 4450 50  0001 C CNN
 F 3 "" H 5850 4450 50  0001 C CNN
@@
 P 5850 3350
 F 0 "H2" H 6050 3300 50  0000 R CNN
-F 1 "M_~SLP" H 5950 3500 50  0000 R CNN
+F 1 "M~SLP" H 5950 3500 50  0000 R CNN
 F 2 "Custom:Mounting_Pad_Signal" H 5850 3500 50  0001 C CNN
 F 3 "" H 5850 3500 50  0001 C CNN
@@
 F 2 "Package_SO:SOIC-16_3.9x9.9mm_P1.27mm" H 2800 2100 50  0001 L CNN
 F 3 "http://www.datasheet5.com/pdf-local-2195953" H 2400 3450 50  0001 C CNN
+F 4 "C84681" H 2750 2650 50  0001 C CNN "LCSC"
 	1    2750 2650
 	1    0    0    -1
@@
 F 2 "Package_TO_SOT_SMD:SOT-23-5" H 1950 6275 50  0001 C CNN
 F 3 "https://www.exar.com/content/document.ashx?id=22106&languageid=1033&type=Datasheet&partnumber=SPX3819&filename=SPX3819.pdf&part=SPX3819" H 1950 5950 50  0001 C CNN
+F 4 "C9055" H 1950 5950 50  0001 C CNN "LCSC"
 	1    1950 5950
 	1    0    0    -1

Commit message: BOM items
Parts:
- C1: Manufacturer Nbr (none) -> TCC0805X7R104K500DT
- C2: Manufacturer Nbr (none) -> CL21A226MQQNNNE
- D1: Manufacturer Nbr (none) -> FC-A2012BK-470H2
- D2: Manufacturer Nbr (none) -> FC-2012UGK-520D5
- J1: Manufacturer Nbr (none) -> C40942
- Q1, Q2: Manufacturer Nbr (none) -> 2SC1623
- R1, R18, R2: Manufacturer Nbr (none) -> 0805W8F1002T5E
- R3, R4: Manufacturer Nbr (none) -> 0805W8J0151T5E
- U1: Manufacturer Nbr (none) -> CH340C
- U3: Manufacturer Nbr (none) -> SPX3819M5-L-3-3/TR
Changed lines of the file:
@@
 F 3 "~" H 7700 1150 50  0001 C CNN
 F 4 "C38522" H 7700 1150 50  0001 C CNN "LCSC"
+F 5 "0805W8F1002T5E" H 7700 1150 50  0001 C CNN "Manufacturer Nbr"
 	1    7700 1150
 	1    0    0    -1
@@
 F 3 "~" H 2250 1800 50  0001 C CNN
 F 4 "C282732" H 2250 1800 50  0001 C CNN "LCSC"
+F 5 "TCC0805X7R104K500DT" H 2250 1800 50  0001 C CNN "Manufacturer Nbr"
 	1    2250 1800
 	1    0    0    -1
@@
 F 3 "~" H 4050 1850 50  0001 C CNN
 F 4 "C5674" H 4050 1850 50  0001 C CNN "LCSC"
+F 5 "CL21A226MQQNNNE" H 4050 1850 50  0001 C CNN "Manufacturer Nbr"
 	1    4050 1850
 	1    0    0    -1
@@
 F 3 "http://www.infineon.com/dgdl/Infineon-BC847SERIES_BC848SERIES_BC849SERIES_BC850SERIES-DS-v01_01-en.pdf?fileId=db3a304314dca389011541d4630a1657" H 4600 2650 50  0001 L CNN
 F 4 "C163753" H 4600 2650 50  0001 C CNN "LCSC"
+F 5 "2SC1623" H 4600 2650 50  0001 C CNN "Manufacturer Nbr"
 	1    4600 2650
 	1    0    0    -1
@@
 F 3 "http://www.infineon.com/dgdl/Infineon-BC847SERIES_BC848SERIES_BC849SERIES_BC850SERIES-DS-v01_01-en.pdf?fileId=db3a304314dca389011541d4630a1657" H 4600 3350 50  0001 L CNN
 F 4 "C163753" H 4600 3350 50  0001 C CNN "LCSC"
+F 5 "2SC1623" H 4600 3350 50  0001 C CNN "Manufacturer Nbr"
 	1    4600 3350
 	1    0    0    1
@@
 F 3 "~" H 4150 2650 50  0001 C CNN
 F 4 "C38522" H 4150 2650 50  0001 C CNN "LCSC"
+F 5 "0805W8F1002T5E" H 4150 2650 50  0001 C CNN "Manufacturer Nbr"
 	1    4150 2650
 	0    -1   -1   0
@@
 F 3 "~" H 4150 3350 50  0001 C CNN
 F 4 "C38522" H 4150 3350 50  0001 C CNN "LCSC"
+F 5 "0805W8F1002T5E" H 4150 3350 50  0001 C CNN "Manufacturer Nbr"
 	1    4150 3350
 	0    1    1    0
@@
 F 3 "~" H 9700 5650 50  0001 C CNN
 F 4 "C84259" H 9700 5650 50  0001 C CNN "LCSC"
+F 5 "FC-A2012BK-470H2" H 9700 5650 50  0001 C CNN "Manufacturer Nbr"
 	1    9700 5650
 	0    -1   -1   0
@@
 F 3 "~" H 9700 5300 50  0001 C CNN
 F 4 "C25283" H 9700 5300 50  0001 C CNN "LCSC"
+F 5 "0805W8J0151T5E" H 9700 5300 50  0001 C CNN "Manufacturer Nbr"
 	1    9700 5300
 	-1   0    0    1
@@
 F 3 "~" H 10700 5650 50  0001 C CNN
 F 4 "C84260" H 10700 5650 50  0001 C CNN "LCSC"
+F 5 "FC-2012UGK-520D5" H 10700 5650 50  0001 C CNN "Manufacturer Nbr"
 	1    10700 5650
 	0    -1   -1   0
@@
 F 3 "~" H 10700 5300 50  0001 C CNN
 F 4 "C25283" H 10700 5300 50  0001 C CNN "LCSC"
+F 5 "0805W8J0151T5E" H 10700 5300 50  0001 C CNN "Manufacturer Nbr"
 	1    10700 5300
 	-1   0    0    1
@@
 F 4 "C40942" H 1100 2100 50  0001 C CNN "LCSC"
 F 5 "2782045" H 1100 2100 50  0001 C CNN "Farnell"
+F 6 "C40942" H 1100 2100 50  0001 C CNN "Manufacturer Nbr"
 	1    1100 2100
 	1    0    0    -1
@@
 F 3 "http://www.datasheet5.com/pdf-local-2195953" H 2400 3450 50  0001 C CNN
 F 4 "C84681" H 2750 2650 50  0001 C CNN "LCSC"
+F 5 "CH340C" H 2750 2650 50  0001 C CNN "Manufacturer Nbr"
 	1    2750 2650
 	1    0    0    -1
@@
 F 3 "https://www.exar.com/content/document.ashx?id=22106&languageid=1033&type=Datasheet&partnumber=SPX3819&filename=SPX3819.pdf&part=SPX3819" H 1950 5950 50  0001 C CNN
 F 4 "C9055" H 1950 5950 50  0001 C CNN "LCSC"
+F 5 "SPX3819M5-L-3-3/TR" H 1950 5950 50  0001 C CNN "Manufacturer Nbr"
 	1    1950 5950
 	1    0    0    -1
