File: robot/Top/Top.sch (KiCad schematic (older format))
At the start: 23 parts, among them J1 Conn_01x02_Male, J2 USB_B_Micro, SW1 SW_DPDT_x2, U1 LD1117S33CTR, U2 MCP73831-2-OT, U3 SSD1306

Commit message: Cleanup, start PDB Front
Parts:
- removed C1: 10µ, symbol Device:C
- removed J2: USB_B_Micro, symbol Connector:USB_B_Micro
- removed TP1, TP2: TestPoint, symbol Connector:TestPoint
- removed U1: LD1117S33CTR, digikey-footprints:SOT-223, symbol dk_PMIC-Voltage-Regulators-Linear:LD1117S33CTR
- added H1: BAT_MON, symbol Custom:MountingPad
- added H2: VBAT_SWITCH, symbol Custom:MountingPad
- added H3: OLED_~RES, symbol Custom:MountingPad
- added H4: OLED_SCL, symbol Custom:MountingPad
- added H5: OLED_SDA, symbol Custom:MountingPad
- added H6, H9: VBUS, symbol Custom:MountingPad
- added H7: 3V3, symbol Custom:MountingPad
- added H8: GND, symbol Custom:MountingPad
Connections:
- net +3V3: now also H7.1 (Pin)
- net BAT_MON: now also H1.1 (Pin)
- net GND: now also H8.1 (Pin)
- net OLED_SCL: now also H4.1 (Pin)
- net OLED_SDA: now also H5.1 (Pin)
- net OLED_~RES: now also H3.1 (Pin)
- net VBUS: now also H6.1 (Pin), H9.1 (Pin); no longer D1.1 (K)
- new net VBAT_SWITCH: D1.1 (K), H2.1 (Pin)
- no-connect marks 2 -> 1
Other:
- note added: "BATTERY SWITCH"
- note removed: "POWER CONVERTOR"
- moved on the sheet: C2, C3, C4, C5, C6, C7, D1, D2, J1, R1, R2, R3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

Commit message: Top PCB
Parts:
- removed H9: VBUS, symbol Custom:MountingPad
- removed TP3: TestPoint, symbol Connector:TestPoint
- added H10: GND, Custom:Mounting_Pad_Power, symbol Custom:MountingPad
- C2, C3, C4, C5, C6, C7: footprint (none) -> Capacitors_SMD:C_1206
- D1: footprint (none) -> Diodes_SMD:D_SOD-123
- D2: footprint (none) -> LEDs:LED_0603
- H1, H3, H4, H5: footprint (none) -> Custom:Mounting_Pad_Signal
- H2, H6, H7, H8: footprint (none) -> Custom:Mounting_Pad_Power
- J1: footprint (none) -> Custom:Conn_Bat
- R1, R2, R3, R4, R5: footprint (none) -> Resistors_SMD:R_1206
- SW1: footprint (none) -> Custom:JS102011SAQN
- U3: footprint (none) -> Custom:SSD1306_OLED
Connections:
- net GND: now also H10.1 (Pin)
Other:
- moved on the sheet: H7, H8

Commit message: Finish Top, remap OLED pins
Parts:
- C2, C3, C4, C5, C6, C7: footprint Capacitors_SMD:C_1206 -> Capacitors_SMD:C_0805
- R1, R2, R3, R4, R5: footprint Resistors_SMD:R_1206 -> Resistors_SMD:R_0805
Changed lines of the file:
@@
 F 0 "R4" H 3920 6096 50  0000 L CNN
 F 1 "5K" H 3920 6005 50  0000 L CNN
-F 2 "Resistors_SMD:R_1206" V 3780 6050 50  0001 C CNN
+F 2 "Resistors_SMD:R_0805" V 3780 6050 50  0001 C CNN
 F 3 "~" H 3850 6050 50  0001 C CNN
 	1    3850 6050
@@
 F 0 "C2" H 5415 5846 50  0000 L CNN
 F 1 "10µ" H 5415 5755 50  0000 L CNN
-F 2 "Capacitors_SMD:C_1206" H 5338 5650 50  0001 C CNN
+F 2 "Capacitors_SMD:C_0805" H 5338 5650 50  0001 C CNN
 F 3 "~" H 5300 5800 50  0001 C CNN
 	1    5300 5800
@@
 F 0 "R3" H 4920 5396 50  0000 L CNN
 F 1 "1K" H 4920 5305 50  0000 L CNN
-F 2 "Resistors_SMD:R_1206" V 4780 5350 50  0001 C CNN
+F 2 "Resistors_SMD:R_0805" V 4780 5350 50  0001 C CNN
 F 3 "~" H 4850 5350 50  0001 C CNN
 	1    4850 5350
@@
 F 0 "R1" H 4720 1946 50  0000 L CNN
 F 1 "100K" H 4720 1855 50  0000 L CNN
-F 2 "Resistors_SMD:R_1206" V 4580 1900 50  0001 C CNN
+F 2 "Resistors_SMD:R_0805" V 4580 1900 50  0001 C CNN
 F 3 "~" H 4650 1900 50  0001 C CNN
 	1    4650 1900
@@
 F 0 "R2" H 4720 2446 50  0000 L CNN
 F 1 "100K" H 4720 2355 50  0000 L CNN
-F 2 "Resistors_SMD:R_1206" V 4580 2400 50  0001 C CNN
+F 2 "Resistors_SMD:R_0805" V 4580 2400 50  0001 C CNN
 F 3 "~" H 4650 2400 50  0001 C CNN
 	1    4650 2400
@@
 F 0 "C3" V 8650 2400 50  0000 C CNN
 F 1 "1µ" V 8750 2650 50  0000 C CNN
-F 2 "Capacitors_SMD:C_1206" H 8738 2400 50  0001 C CNN
+F 2 "Capacitors_SMD:C_0805" H 8738 2400 50  0001 C CNN
 F 3 "~" H 8700 2550 50  0001 C CNN
 	1    8700 2550
@@
 F 0 "C4" V 8650 2700 50  0000 C CNN
 F 1 "1µ" V 8750 2950 50  0000 C CNN
-F 2 "Capacitors_SMD:C_1206" H 8738 2700 50  0001 C CNN
+F 2 "Capacitors_SMD:C_0805" H 8738 2700 50  0001 C CNN
 F 3 "~" H 8700 2850 50  0001 C CNN
 	1    8700 2850
@@
 F 0 "C5" V 8650 3000 50  0000 C CNN
 F 1 "1µ" V 8750 3250 50  0000 C CNN
-F 2 "Capacitors_SMD:C_1206" H 8738 3000 50  0001 C CNN
+F 2 "Capacitors_SMD:C_0805" H 8738 3000 50  0001 C CNN
 F 3 "~" H 8700 3150 50  0001 C CNN
 	1    8700 3150
@@
 F 0 "C6" V 8650 4200 50  0000 C CNN
 F 1 "4.7µ" V 8750 4500 50  0000 C CNN
-F 2 "Capacitors_SMD:C_1206" H 8738 4200 50  0001 C CNN
+F 2 "Capacitors_SMD:C_0805" H 8738 4200 50  0001 C CNN
 F 3 "~" H 8700 4350 50  0001 C CNN
 	1    8700 4350
@@
 F 0 "C7" V 8750 4750 50  0000 C CNN
 F 1 "4.7µ" V 8650 4450 50  0000 C CNN
-F 2 "Capacitors_SMD:C_1206" H 8738 4450 50  0001 C CNN
+F 2 "Capacitors_SMD:C_0805" H 8738 4450 50  0001 C CNN
 F 3 "~" H 8700 4600 50  0001 C CNN
 	1    8700 4600
@@
 F 0 "R5" V 8750 4350 50  0000 C CNN
 F 1 "330k" V 8650 3950 50  0000 C CNN
-F 2 "Resistors_SMD:R_1206" V 8630 4150 50  0001 C CNN
+F 2 "Resistors_SMD:R_0805" V 8630 4150 50  0001 C CNN
 F 3 "~" H 8700 4150 50  0001 C CNN
 	1    8700 4150
