File: robot/Top/Top.kicad_pcb (KiCad board)
At the start: 2 copper layers, 40 x 40 mm, 26 parts, among them J1 Conn_01x02_Male, SW1 SW_DPDT_x2, U2 MCP73831-2-OT, U3 SSD1306

Commit message: Small changes to top, step
Parts:
- moved D1 0.45 mm to (150.5, 125.5)
Changed lines of the file:
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@@
     (thickness 1.6)
     (drawings 13)
-    (tracks 137)
+    (tracks 136)
     (zones 0)
     (modules 26)
@@
   )
   (setup
-    (last_trace_width 0.2)
+    (last_trace_width 0.4)
     (user_trace_width 0.2)
     (user_trace_width 0.3)
@@
   )
   (module Diodes_SMD:D_SOD-123 (layer B.Cu)
-    (at 150.5 125.9)
+    (at 150.5 125.45)
     (descr SOD-123)
     (tags SOD-123)
@@
   (segment (start 132.3 117) (end 132.8 117.5) (width 0.4) (layer B.Cu) (net 2))
   (segment (start 132.3 113.3) (end 132.3 117) (width 0.4) (layer B.Cu) (net 2))
-  (segment (start 132.8 117.5) (end 132.8 121.8) (width 0.4) (layer B.Cu) (net 2))
-  (segment (start 132.8 121.8) (end 144.5 133.5) (width 0.4) (layer B.Cu) (net 2))
   (segment (start 153 129.4) (end 153 128.75) (width 0.4) (layer B.Cu) (net 2))
-  (segment (start 148.9 133.5) (end 153 129.4) (width 0.4) (layer B.Cu) (net 2))
-  (segment (start 144.5 133.5) (end 148.9 133.5) (width 0.4) (layer B.Cu) (net 2))
   (segment (start 132.3 113.3) (end 132.3 112.3) (width 0.2) (layer B.Cu) (net 2))
   (segment (start 143.5 102) (end 145.45 100.05) (width 0.2) (layer B.Cu) (net 2))
@@
   (segment (start 132.07 108.1) (end 131.8 108.37) (width 0.2) (layer B.Cu) (net 2))
   (segment (start 136.420002 108.1) (end 132.07 108.1) (width 0.2) (layer B.Cu) (net 2))
+  (segment (start 132.8 121.8) (end 144.5 133.5) (width 0.4) (layer B.Cu) (net 2))
+  (segment (start 132.8 117.5) (end 132.8 121.8) (width 0.4) (layer B.Cu) (net 2))
+  (segment (start 144.5 133.5) (end 148.9 133.5) (width 0.4) (layer B.Cu) (net 2))
+  (segment (start 148.9 133.5) (end 153 129.4) (width 0.4) (layer B.Cu) (net 2))
   (segment (start 168.5 115.25) (end 169.5 115.25) (width 0.2) (layer B.Cu) (net 3))
   (segment (start 165.15 113.24) (end 166.49 113.24) (width 0.2) (layer B.Cu) (net 3))
@@
   (segment (start 167.25 103.75) (end 167.125 103.75) (width 0.2) (layer B.Cu) (net 9))
   (via (at 135.2 97.95) (size 1) (drill 0.5) (layers F.Cu B.Cu) (net 10))
-  (via (at 148.85 125.9) (size 1) (drill 0.5) (layers F.Cu B.Cu) (net 10))
   (segment (start 135.2 97.95) (end 135.2 99.2) (width 0.4) (layer F.Cu) (net 10))
-  (segment (start 135.2 99.2) (end 137.1 101.1) (width 0.4) (layer F.Cu) (net 10))
-  (via (at 137.55 110.9) (size 1) (drill 0.5) (layers F.Cu B.Cu) (net 10))
-  (segment (start 137.1 110.45) (end 137.55 110.9) (width 0.4) (layer F.Cu) (net 10))
-  (segment (start 137.1 110.35) (end 137.1 110.45) (width 0.4) (layer F.Cu) (net 10))
-  (segment (start 137.1 101.1) (end 137.1 110.35) (width 0.4) (layer F.Cu) (net 10))
-  (segment (start 148 125.9) (end 148.85 125.9) (width 0.4) (layer B.Cu) (net 10))
-  (segment (start 137.55 115.45) (end 148 125.9) (width 0.4) (layer B.Cu) (net 10))
-  (segment (start 137.55 110.9) (end 137.55 115.45) (width 0.4) (layer B.Cu) (net 10))
-  (segment (start 150.5 127.55) (end 152.15 125.9) (width 0.4) (layer B.Cu) (net 11))
-  (segment (start 150.5 128.75) (end 150.5 127.55) (width 0.4) (layer B.Cu) (net 11))
+  (segment (start 135.2 99.2) (end 137.45 101.45) (width 0.4) (layer F.Cu) (net 10))
+  (via (at 137.45 113.3) (size 1) (drill 0.5) (layers F.Cu B.Cu) (net 10))
+  (segment (start 137.45 101.45) (end 137.45 113.3) (width 0.4) (layer F.Cu) (net 10))
+  (segment (start 137.45 113.3) (end 137.45 115.35) (width 0.4) (layer B.Cu) (net 10))
+  (via (at 148.85 125.45) (size 1) (drill 0.5) (layers F.Cu B.Cu) (net 10))
+  (segment (start 148 125.45) (end 148.85 125.45) (width 0.4) (layer B.Cu) (net 10))
+  (segment (start 147.55 125.45) (end 148 125.45) (width 0.4) (layer B.Cu) (net 10))
+  (segment (start 137.45 115.35) (end 147.55 125.45) (width 0.4) (layer B.Cu) (net 10))
+  (segment (start 150.5 127.1) (end 152.15 125.45) (width 0.4) (layer B.Cu) (net 11))
+  (segment (start 150.5 128.75) (end 150.5 127.1) (width 0.4) (layer B.Cu) (net 11))
   (segment (start 131.8 106.695) (end 133.5 104.995) (width 0.4) (layer B.Cu) (net 12))
   (segment (start 131.8 106.9) (end 131.8 106.695) (width 0.4) (layer B.Cu) (net 12))

Commit message: Layout changes, new footprints, added Side PCB
Parts:
- H2: value VBS -> VSW
- H6: value VBUS -> VBS
Changed lines of the file:
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@@
-(kicad_pcb (version 20171130) (host pcbnew "(5.1.2)-1")
+(kicad_pcb (version 20171130) (host pcbnew "(5.1.4)-1")
   (general
     (thickness 1.6)
@@
   )
   (setup
-    (last_trace_width 0.4)
+    (last_trace_width 0.2)
     (user_trace_width 0.2)
     (user_trace_width 0.3)
@@
       (effects (font (size 0.9 1) (thickness 0.15)) (justify mirror))
     )
-    (fp_text value VBUS (at 0 3.3) (layer B.SilkS)
+    (fp_text value VBS (at 0 3.3) (layer B.SilkS)
       (effects (font (size 0.9 1) (thickness 0.15)) (justify mirror))
     )
@@
       (effects (font (size 0.9 1) (thickness 0.15)) (justify mirror))
     )
-    (fp_text value VBS (at 0 3.3) (layer B.SilkS)
-      (effects (font (size 0.9 1) (thickness 0.15)) (justify mirror))
-    )
+    (fp_text value VSW (at 0 3.3) (layer B.SilkS)
+      (effects (font (size 0.9 1) (thickness 0.15)) (justify mirror))
+    )

Commit message: Top changes
Parts:
- moved SW1 1.80 mm to (150.5, 130.6)
- moved D1 1.75 mm to (150.5, 127.2)
Routing:
- net /VBAT_SWITCH: track 33.9 -> 34.9 mm, vias 3 -> 2
- net GND: vias 11 -> 12
Changed lines of the file:
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@@
     (46 B.CrtYd user)
     (47 F.CrtYd user)
-    (48 B.Fab user hide)
-    (49 F.Fab user hide)
+    (48 B.Fab user)
+    (49 F.Fab user)
   )
   (setup
-    (last_trace_width 0.2)
+    (last_trace_width 0.4)
     (user_trace_width 0.2)
     (user_trace_width 0.3)
@@
   )
   (module Diodes_SMD:D_SOD-123 (layer B.Cu)
-    (at 150.5 125.45)
+    (at 150.5 127.2)
     (descr SOD-123)
     (tags SOD-123)
@@
   )
   (module Custom:JS102011SAQN (layer B.Cu)
-    (at 150.5 128.75 180)
+    (at 150.5 130.55 180)
     (fp_text reference SW1 (at 0.2 -2.7 180) (layer B.SilkS)
       (effects (font (size 0.9 1) (thickness 0.15)) (justify mirror))
@@
     (pad 1 smd rect (at -2.5 0 180) (size 1.2 2.5) (layers B.Cu B.Paste B.Mask)
       (net 2 +BATT))
+    (model C:/Users/tinus/Documents/Projects_on_GitHub/kicad_custom_libraries/Custom.3dshapes/JS102011SAQN.step
+      (at (xyz 0 0 0))
+      (scale (xyz 1 1 1))
+      (rotate (xyz 0 0 0))
+    )
   )
   (module Custom:Conn_Bat (layer B.Cu)
@@
   (via (at 141.7 100.65) (size 0.8) (drill 0.4) (layers F.Cu B.Cu) (net 1))
   (via (at 150.5 115.5) (size 1) (drill 0.5) (layers F.Cu B.Cu) (net 1))
+  (via (at 132.55 123.75) (size 1) (drill 0.5) (layers F.Cu B.Cu) (net 1))
   (segment (start 145.45 100.05) (end 145.45 99.75) (width 0.2) (layer B.Cu) (net 2))
   (segment (start 131.8 112.8) (end 132.3 113.3) (width 0.4) (layer B.Cu) (net 2))
@@
   (segment (start 132.3 117) (end 132.8 117.5) (width 0.4) (layer B.Cu) (net 2))
   (segment (start 132.3 113.3) (end 132.3 117) (width 0.4) (layer B.Cu) (net 2))
-  (segment (start 153 129.4) (end 153 128.75) (width 0.4) (layer B.Cu) (net 2))
   (segment (start 132.3 113.3) (end 132.3 112.3) (width 0.2) (layer B.Cu) (net 2))
   (segment (start 143.5 102) (end 145.45 100.05) (width 0.2) (layer B.Cu) (net 2))
@@
   (segment (start 132.07 108.1) (end 131.8 108.37) (width 0.2) (layer B.Cu) (net 2))
   (segment (start 136.420002 108.1) (end 132.07 108.1) (width 0.2) (layer B.Cu) (net 2))
-  (segment (start 132.8 121.8) (end 144.5 133.5) (width 0.4) (layer B.Cu) (net 2))
-  (segment (start 132.8 117.5) (end 132.8 121.8) (width 0.4) (layer B.Cu) (net 2))
-  (segment (start 144.5 133.5) (end 148.9 133.5) (width 0.4) (layer B.Cu) (net 2))
-  (segment (start 148.9 133.5) (end 153 129.4) (width 0.4) (layer B.Cu) (net 2))
+  (segment (start 132.8 117.5) (end 132.8 120.9) (width 0.4) (layer B.Cu) (net 2))
+  (segment (start 132.8 120.9) (end 146.5 134.6) (width 0.4) (layer B.Cu) (net 2))
+  (segment (start 153 131.2) (end 153 130.55) (width 0.4) (layer B.Cu) (net 2))
+  (segment (start 149.6 134.6) (end 153 131.2) (width 0.4) (layer B.Cu) (net 2))
+  (segment (start 146.5 134.6) (end 149.6 134.6) (width 0.4) (layer B.Cu) (net 2))
   (segment (start 168.5 115.25) (end 169.5 115.25) (width 0.2) (layer B.Cu) (net 3))
   (segment (start 165.15 113.24) (end 166.49 113.24) (width 0.2) (layer B.Cu) (net 3))
@@
   (via (at 137.45 113.3) (size 1) (drill 0.5) (layers F.Cu B.Cu) (net 10))
   (segment (start 137.45 101.45) (end 137.45 113.3) (width 0.4) (layer F.Cu) (net 10))
-  (segment (start 137.45 113.3) (end 137.45 115.35) (width 0.4) (layer B.Cu) (net 10))
-  (via (at 148.85 125.45) (size 1) (drill 0.5) (layers F.Cu B.Cu) (net 10))
-  (segment (start 148 125.45) (end 148.85 125.45) (width 0.4) (layer B.Cu) (net 10))
-  (segment (start 147.55 125.45) (end 148 125.45) (width 0.4) (layer B.Cu) (net 10))
-  (segment (start 137.45 115.35) (end 147.55 125.45) (width 0.4) (layer B.Cu) (net 10))
-  (segment (start 150.5 127.1) (end 152.15 125.45) (width 0.4) (layer B.Cu) (net 11))
-  (segment (start 150.5 128.75) (end 150.5 127.1) (width 0.4) (layer B.Cu) (net 11))
+  (segment (start 148.85 127.05) (end 148.85 127.2) (width 0.4) (layer B.Cu) (net 10))
+  (segment (start 137.45 115.65) (end 148.85 127.05) (width 0.4) (layer B.Cu) (net 10))
+  (segment (start 137.45 113.3) (end 137.45 115.65) (width 0.4) (layer B.Cu) (net 10))
+  (segment (start 152.15 128.25) (end 152.15 127.2) (width 0.4) (layer B.Cu) (net 11))
+  (segment (start 150.5 130.55) (end 150.5 129.9) (width 0.4) (layer B.Cu) (net 11))
+  (segment (start 150.5 129.9) (end 152.15 128.25) (width 0.4) (layer B.Cu) (net 11))
   (segment (start 131.8 106.695) (end 133.5 104.995) (width 0.4) (layer B.Cu) (net 12))
   (segment (start 131.8 106.9) (end 131.8 106.695) (width 0.4) (layer B.Cu) (net 12))
