File: robot/Bottom/Bottom.sch (KiCad schematic (older format))
At the start: 35 parts, among them M1 Stepper_Motor_bipolar, M2 Stepper_Motor_bipolar, U1 GP2S60, U2 GP2S60, U7 DRV8833PWP, U8 DRV8833PWP

Commit message: Cleanup, start PDB Front
Parts:
- added H16, H17: GND_TOUCH, symbol Custom:MountingPad
Connections:
- net GND: now also H16.1 (Pin), H17.1 (Pin)
Other:
- note added: "PADS TO DRAG ON FLOOR"
Changed lines of the file:
@@
 EESchema Schematic File Version 4
+LIBS:Bottom-cache
 EELAYER 29 0
 EELAYER END
@@
 encoding utf-8
 Sheet 1 1
-Title ""
-Date ""
+Title "Motor and Edge detection"
+Date "2019-09-06"
 Rev ""
 Comp ""
@@
 	9250 1400 9250 1300
 $Comp
+L Custom:MountingPad H17
+U 1 1 5D91B15C
+P 4350 7050
+F 0 "H17" H 4500 7000 50  0000 R CNN
+F 1 "GND_TOUCH" H 4850 7100 50  0000 R CNN
+F 2 "" H 4350 7200 50  0001 C CNN
+F 3 "" H 4350 7200 50  0001 C CNN
+	1    4350 7050
+	1    0    0    -1
+$EndComp
+$Comp
+L Custom:MountingPad H16
+U 1 1 5D91B695
+P 4150 7050
+F 0 "H16" H 4100 7000 50  0000 R CNN
+F 1 "GND_TOUCH" H 4100 7100 50  0000 R CNN
+F 2 "" H 4150 7200 50  0001 C CNN
+F 3 "" H 4150 7200 50  0001 C CNN
+	1    4150 7050
+	1    0    0    -1
+$EndComp
+$Comp
+L power:GND #PWR011
+U 1 1 5D932EB6
+P 4150 7450
+F 0 "#PWR011" H 4150 7200 50  0001 C CNN
+F 1 "GND" H 4155 7277 50  0000 C CNN
+F 2 "" H 4150 7450 50  0001 C CNN
+F 3 "" H 4150 7450 50  0001 C CNN
+	1    4150 7450
+	1    0    0    -1
+$EndComp
+$Comp
+L power:GND #PWR012
+U 1 1 5D9331C8
+P 4350 7450
+F 0 "#PWR012" H 4350 7200 50  0001 C CNN
+F 1 "GND" H 4355 7277 50  0000 C CNN
+F 2 "" H 4350 7450 50  0001 C CNN
+F 3 "" H 4350 7450 50  0001 C CNN
+	1    4350 7450
+	1    0    0    -1
+$EndComp
+Wire Wire Line
+	4150 7350 4150 7450
+$Comp
 L power:PWR_FLAG #FLG01
-U 1 1 5D7CE852
-P 10100 1300
-F 0 "#FLG01" H 10100 1375 50  0001 C CNN
-F 1 "PWR_FLAG" H 10100 1473 50  0000 C CNN
-F 2 "" H 10100 1300 50  0001 C CNN
-F 3 "~" H 10100 1300 50  0001 C CNN
-	1    10100 1300
-	-1   0    0    1
+U 1 1 5D948697
+P 10100 1150
+F 0 "#FLG01" H 10100 1225 50  0001 C CNN
+F 1 "PWR_FLAG" H 10100 1323 50  0000 C CNN
+F 2 "" H 10100 1150 50  0001 C CNN
+F 3 "~" H 10100 1150 50  0001 C CNN
+	1    10100 1150
+	1    0    0    -1
 $EndComp
 $Comp
 L power:PWR_FLAG #FLG02
-U 1 1 5D7CF32D
-P 10500 1450
-F 0 "#FLG02" H 10500 1525 50  0001 C CNN
-F 1 "PWR_FLAG" H 10500 1623 50  0000 C CNN
-F 2 "" H 10500 1450 50  0001 C CNN
-F 3 "~" H 10500 1450 50  0001 C CNN
-	1    10500 1450
+U 1 1 5D948E91
+P 10400 1150
+F 0 "#FLG02" H 10400 1225 50  0001 C CNN
+F 1 "PWR_FLAG" H 10400 1323 50  0000 C CNN
+F 2 "" H 10400 1150 50  0001 C CNN
+F 3 "~" H 10400 1150 50  0001 C CNN
+	1    10400 1150
+	-1   0    0    1
+$EndComp
+$Comp
+L power:GND #PWR010
+U 1 1 5D949163
+P 10100 1250
+F 0 "#PWR010" H 10100 1000 50  0001 C CNN
+F 1 "GND" H 10105 1077 50  0000 C CNN
+F 2 "" H 10100 1250 50  0001 C CNN
+F 3 "" H 10100 1250 50  0001 C CNN
+	1    10100 1250
 	1    0    0    -1
 $EndComp
 $Comp
 L power:+3V3 #PWR09
-U 1 1 5D7CF89A
-P 10100 1200
-F 0 "#PWR09" H 10100 1050 50  0001 C CNN
-F 1 "+3V3" H 10115 1373 50  0000 C CNN
-F 2 "" H 10100 1200 50  0001 C CNN
-F 3 "" H 10100 1200 50  0001 C CNN
-	1    10100 1200
-	1    0    0    -1
-$EndComp
-$Comp
-L power:GND #PWR010
-U 1 1 5D7CFB04
-P 10500 1550
-F 0 "#PWR010" H 10500 1300 50  0001 C CNN
-F 1 "GND" H 10505 1377 50  0000 C CNN
-F 2 "" H 10500 1550 50  0001 C CNN
-F 3 "" H 10500 1550 50  0001 C CNN
-	1    10500 1550
-	1    0    0    -1
-$EndComp
-Wire Wire Line
-	10100 1200 10100 1300
-Wire Wire Line
-	10500 1450 10500 1550
+U 1 1 5D949502
+P 10400 1050
+F 0 "#PWR09" H 10400 900 50  0001 C CNN
+F 1 "+3V3" H 10415 1223 50  0000 C CNN
+F 2 "" H 10400 1050 50  0001 C CNN
+F 3 "" H 10400 1050 50  0001 C CNN
+	1    10400 1050
+	1    0    0    -1
+$EndComp
+Wire Wire Line
+	10100 1150 10100 1250
+Wire Wire Line
+	10400 1050 10400 1150
+Wire Wire Line
+	4350 7350 4350 7450
+Text Notes 3800 6750 0    50   ~ 0
+PADS TO DRAG ON FLOOR
 $EndSCHEMATC

Commit message: Bottom
Parts:
- C10, C11, C12, C13, C8, C9: footprint (none) -> Capacitors_SMD:C_1206
- H1: value A1 -> M1A1; footprint (none) -> Custom:Mounting_Pad_Signal
- H10: value B2 -> M2B2; footprint (none) -> Custom:Mounting_Pad_Signal
- H11: value M_~SLEEP -> M_~SLP; footprint (none) -> Custom:Mounting_Pad_Signal
- H12, H13, H14, H15, H16, H17: footprint (none) -> Custom:Mounting_Pad_Power
- H2: value A2 -> M1A2; footprint (none) -> Custom:Mounting_Pad_Signal
- H3: value B1 -> M1B1; footprint (none) -> Custom:Mounting_Pad_Signal
- H4: value B2 -> M1B2; footprint (none) -> Custom:Mounting_Pad_Signal
- H5: value ED_OUT1 -> ED1; footprint (none) -> Custom:Mounting_Pad_Signal
- H6: value ED_OUT2 -> ED2; footprint (none) -> Custom:Mounting_Pad_Signal
- H7: value A1 -> M2A1; footprint (none) -> Custom:Mounting_Pad_Signal
- H8: value A2 -> M2A2; footprint (none) -> Custom:Mounting_Pad_Signal
- H9: value B1 -> M2B1; footprint (none) -> Custom:Mounting_Pad_Signal
- R1, R11, R12, R13, R14, R2, R3, R4: footprint (none) -> Resistors_SMD:R_1206
- U1, U2: footprint (none) -> Custom:GP2S60_ReverseMount
Other:
- moved on the sheet: H11
Changed lines of the file:
@@
 F 0 "C9" H 3015 1696 50  0000 L CNN
 F 1 "2.2µ" H 3015 1605 50  0000 L CNN
-F 2 "" H 2938 1500 50  0001 C CNN
+F 2 "Capacitors_SMD:C_1206" H 2938 1500 50  0001 C CNN
 F 3 "~" H 2900 1650 50  0001 C CNN
 	1    2900 1650
@@
 F 0 "C8" H 1865 1696 50  0000 L CNN
 F 1 "0.01µ" H 1865 1605 50  0000 L CNN
-F 2 "" H 1788 1500 50  0001 C CNN
+F 2 "Capacitors_SMD:C_1206" H 1788 1500 50  0001 C CNN
 F 3 "~" H 1750 1650 50  0001 C CNN
 	1    1750 1650
@@
 F 0 "C10" H 3815 1696 50  0000 L CNN
 F 1 "10µ" H 3815 1605 50  0000 L CNN
-F 2 "" H 3738 1500 50  0001 C CNN
+F 2 "Capacitors_SMD:C_1206" H 3738 1500 50  0001 C CNN
 F 3 "~" H 3700 1650 50  0001 C CNN
 	1    3700 1650
@@
 F 0 "R11" H 1370 2796 50  0000 L CNN
 F 1 "0.8" H 1370 2705 50  0000 L CNN
-F 2 "" V 1230 2750 50  0001 C CNN
+F 2 "Resistors_SMD:R_1206" V 1230 2750 50  0001 C CNN
 F 3 "~" H 1300 2750 50  0001 C CNN
 	1    1300 2750
@@
 F 0 "R12" H 1720 2796 50  0000 L CNN
 F 1 "0.8" H 1720 2705 50  0000 L CNN
-F 2 "" V 1580 2750 50  0001 C CNN
+F 2 "Resistors_SMD:R_1206" V 1580 2750 50  0001 C CNN
 F 3 "~" H 1650 2750 50  0001 C CNN
 	1    1650 2750
@@
 F 0 "C12" H 3015 4296 50  0000 L CNN
 F 1 "2.2µ" H 3015 4205 50  0000 L CNN
-F 2 "" H 2938 4100 50  0001 C CNN
+F 2 "Capacitors_SMD:C_1206" H 2938 4100 50  0001 C CNN
 F 3 "~" H 2900 4250 50  0001 C CNN
 	1    2900 4250
@@
 F 0 "C11" H 1865 4296 50  0000 L CNN
 F 1 "0.01µ" H 1865 4205 50  0000 L CNN
-F 2 "" H 1788 4100 50  0001 C CNN
+F 2 "Capacitors_SMD:C_1206" H 1788 4100 50  0001 C CNN
 F 3 "~" H 1750 4250 50  0001 C CNN
 	1    1750 4250
@@
 F 0 "C13" H 3815 4296 50  0000 L CNN
 F 1 "10µ" H 3815 4205 50  0000 L CNN
-F 2 "" H 3738 4100 50  0001 C CNN
+F 2 "Capacitors_SMD:C_1206" H 3738 4100 50  0001 C CNN
 F 3 "~" H 3700 4250 50  0001 C CNN
 	1    3700 4250
@@
 F 0 "R13" H 1370 5396 50  0000 L CNN
 F 1 "0.8" H 1370 5305 50  0000 L CNN
-F 2 "" V 1230 5350 50  0001 C CNN
+F 2 "Resistors_SMD:R_1206" V 1230 5350 50  0001 C CNN
 F 3 "~" H 1300 5350 50  0001 C CNN
 	1    1300 5350
@@
 F 0 "R14" H 1720 5396 50  0000 L CNN
 F 1 "0.8" H 1720 5305 50  0000 L CNN
-F 2 "" V 1580 5350 50  0001 C CNN
+F 2 "Resistors_SMD:R_1206" V 1580 5350 50  0001 C CNN
 F 3 "~" H 1650 5350 50  0001 C CNN
 	1    1650 5350
@@
 F 0 "U1" H 8178 4096 50  0000 L CNN
 F 1 "GP2S60" H 8178 4005 50  0000 L CNN
-F 2 "" H 7750 4050 50  0001 C CNN
+F 2 "Custom:GP2S60_ReverseMount" H 7750 4050 50  0001 C CNN
 F 3 "" H 7750 4050 50  0001 C CNN
 	1    7750 4050
@@
 F 0 "R2" H 8020 3346 50  0000 L CNN
 F 1 "120" H 8020 3255 50  0000 L CNN
-F 2 "" V 7880 3300 50  0001 C CNN
+F 2 "Resistors_SMD:R_1206" V 7880 3300 50  0001 C CNN
 F 3 "~" H 7950 3300 50  0001 C CNN
 	1    7950 3300
@@
 F 0 "R1" H 7620 3346 50  0000 L CNN
 F 1 "10k" H 7620 3255 50  0000 L CNN
-F 2 "" V 7480 3300 50  0001 C CNN
+F 2 "Resistors_SMD:R_1206" V 7480 3300 50  0001 C CNN
 F 3 "~" H 7550 3300 50  0001 C CNN
 	1    7550 3300
@@
 F 0 "U2" H 9978 4096 50  0000 L CNN
 F 1 "GP2S60" H 9978 4005 50  0000 L CNN
-F 2 "" H 9550 4050 50  0001 C CNN
+F 2 "Custom:GP2S60_ReverseMount" H 9550 4050 50  0001 C CNN
 F 3 "" H 9550 4050 50  0001 C CNN
 	1    9550 4050
@@
 F 0 "R4" H 9820 3346 50  0000 L CNN
 F 1 "120" H 9820 3255 50  0000 L CNN
-F 2 "" V 9680 3300 50  0001 C CNN
+F 2 "Resistors_SMD:R_1206" V 9680 3300 50  0001 C CNN
 F 3 "~" H 9750 3300 50  0001 C CNN
 	1    9750 3300
@@
 F 0 "R3" H 9420 3346 50  0000 L CNN
 F 1 "10k" H 9420 3255 50  0000 L CNN
-F 2 "" V 9280 3300 50  0001 C CNN
+F 2 "Resistors_SMD:R_1206" V 9280 3300 50  0001 C CNN
 F 3 "~" H 9350 3300 50  0001 C CNN
 	1    9350 3300
@@
 P 4400 1650
 F 0 "H1" H 4550 1600 50  0000 R CNN
-F 1 "A1" H 4550 1700 50  0000 R CNN
-F 2 "" H 4400 1800 50  0001 C CNN
+F 1 "M1A1" H 4500 1800 50  0000 R CNN
+F 2 "Custom:Mounting_Pad_Signal" H 4400 1800 50  0001 C CNN
 F 3 "" H 4400 1800 50  0001 C CNN
 	1    4400 1650
@@
 P 4650 1650
 F 0 "H2" H 4800 1600 50  0000 R CNN
-F 1 "A2" H 4800 1700 50  0000 R CNN
-F 2 "" H 4650 1800 50  0001 C CNN
+F 1 "M1A2" H 4750 1800 50  0000 R CNN
+F 2 "Custom:Mounting_Pad_Signal" H 4650 1800 50  0001 C CNN
 F 3 "" H 4650 1800 50  0001 C CNN
 	1    4650 1650
@@
 P 4900 1650
 F 0 "H3" H 5050 1600 50  0000 R CNN
-F 1 "B1" H 5050 1700 50  0000 R CNN
-F 2 "" H 4900 1800 50  0001 C CNN
+F 1 "M1B1" H 5000 1800 50  0000 R CNN
+F 2 "Custom:Mounting_Pad_Signal" H 4900 1800 50  0001 C CNN
 F 3 "" H 4900 1800 50  0001 C CNN
 	1    4900 1650
@@
 P 5150 1650
 F 0 "H4" H 5300 1600 50  0000 R CNN
-F 1 "B2" H 5300 1700 50  0000 R CNN
-F 2 "" H 5150 1800 50  0001 C CNN
+F 1 "M1B2" H 5250 1800 50  0000 R CNN
+F 2 "Custom:Mounting_Pad_Signal" H 5150 1800 50  0001 C CNN
 F 3 "" H 5150 1800 50  0001 C CNN
 	1    5150 1650
@@
 L Custom:MountingPad H11
 U 1 1 5D743E3A
-P 3000 7300
-F 0 "H11" H 2912 7140 50  0000 R CNN
-F 1 "M_~SLEEP" H 2912 7238 50  0000 R CNN
-F 2 "" H 3000 7450 50  0001 C CNN
-F 3 "" H 3000 7450 50  0001 C CNN
-	1    3000 7300
-	-1   0    0    1
-$EndComp
-Wire Wire Line
-	3000 7000 3000 6900
-Text Label 2850 6800 2    50   ~ 0
+P 6200 1650
+F 0 "H11" H 6112 1490 50  0000 R CNN
+F 1 "M_~SLP" H 6112 1588 50  0000 R CNN
+F 2 "Custom:Mounting_Pad_Signal" H 6200 1800 50  0001 C CNN
+F 3 "" H 6200 1800 50  0001 C CNN
+	1    6200 1650
+	-1   0    0    1
+$EndComp
+Wire Wire Line
+	6200 1350 6200 1250
+Text Label 6050 1150 2    50   ~ 0
 M2_~SLEEP
-Text Label 2850 6900 2    50   ~ 0
+Text Label 6050 1250 2    50   ~ 0
 M1_~SLEEP
 Wire Wire Line
-	2850 6800 3000 6800
-Wire Wire Line
-	2850 6900 3000 6900
-Connection ~ 3000 6900
-Wire Wire Line
-	3000 6900 3000 6800
+	6050 1150 6200 1150
+Wire Wire Line
+	6050 1250 6200 1250
+Connection ~ 6200 1250
+Wire Wire Line
+	6200 1250 6200 1150
 $Comp
 L Custom:MountingPad H7
@@
 P 4400 4250
 F 0 "H7" H 4550 4200 50  0000 R CNN
-F 1 "A1" H 4550 4300 50  0000 R CNN
-F 2 "" H 4400 4400 50  0001 C CNN
+F 1 "M2A1" H 4500 4400 50  0000 R CNN
+F 2 "Custom:Mounting_Pad_Signal" H 4400 4400 50  0001 C CNN
 F 3 "" H 4400 4400 50  0001 C CNN
 	1    4400 4250
@@
 P 4650 4250
 F 0 "H8" H 4800 4200 50  0000 R CNN
-F 1 "A2" H 4800 4300 50  0000 R CNN
-F 2 "" H 4650 4400 50  0001 C CNN
+F 1 "M2A2" H 4750 4400 50  0000 R CNN
+F 2 "Custom:Mounting_Pad_Signal" H 4650 4400 50  0001 C CNN
 F 3 "" H 4650 4400 50  0001 C CNN
 	1    4650 4250
@@
 P 4900 4250
 F 0 "H9" H 5050 4200 50  0000 R CNN
-F 1 "B1" H 5050 4300 50  0000 R CNN
-F 2 "" H 4900 4400 50  0001 C CNN
+F 1 "M2B1" H 5000 4400 50  0000 R CNN
+F 2 "Custom:Mounting_Pad_Signal" H 4900 4400 50  0001 C CNN
 F 3 "" H 4900 4400 50  0001 C CNN
 	1    4900 4250
@@
 P 5150 4250
 F 0 "H10" H 5300 4200 50  0000 R CNN
-F 1 "B2" H 5300 4300 50  0000 R CNN
-F 2 "" H 5150 4400 50  0001 C CNN
+F 1 "M2B2" H 5250 4400 50  0000 R CNN
+F 2 "Custom:Mounting_Pad_Signal" H 5150 4400 50  0001 C CNN
 F 3 "" H 5150 4400 50  0001 C CNN
 	1    5150 4250
@@
 P 7100 3950
 F 0 "H5" H 7250 3900 50  0000 R CNN
-F 1 "ED_OUT1" H 7500 4000 50  0000 R CNN
-F 2 "" H 7100 4100 50  0001 C CNN
+F 1 "ED1" H 7300 4000 50  0000 R CNN
+F 2 "Custom:Mounting_Pad_Signal" H 7100 4100 50  0001 C CNN
 F 3 "" H 7100 4100 50  0001 C CNN
 	1    7100 3950
@@
 P 8900 3950
 F 0 "H6" H 9050 3900 50  0000 R CNN
-F 1 "ED_OUT2" H 9300 4000 50  0000 R CNN
-F 2 "" H 8900 4100 50  0001 C CNN
+F 1 "ED2" H 9100 4000 50  0000 R CNN
+F 2 "Custom:Mounting_Pad_Signal" H 8900 4100 50  0001 C CNN
 F 3 "" H 8900 4100 50  0001 C CNN
 	1    8900 3950
@@
 F 0 "H12" H 8250 1650 50  0000 R CNN
 F 1 "3V3" H 8300 1750 50  0000 R CNN
-F 2 "" H 8100 1850 50  0001 C CNN
+F 2 "Custom:Mounting_Pad_Power" H 8100 1850 50  0001 C CNN
 F 3 "" H 8100 1850 50  0001 C CNN
 	1    8100 1700
@@
 F 0 "H13" H 8500 1750 50  0000 R CNN
 F 1 "GND" H 8550 1650 50  0000 R CNN
-F 2 "" H 8350 1850 50  0001 C CNN
+F 2 "Custom:Mounting_Pad_Power" H 8350 1850 50  0001 C CNN
 F 3 "" H 8350 1850 50  0001 C CNN
 	1    8350 1700
@@
 F 0 "H14" H 8950 1750 50  0000 R CNN
 F 1 "GND" H 8950 1650 50  0000 R CNN
-F 2 "" H 9000 1850 50  0001 C CNN
+F 2 "Custom:Mounting_Pad_Power" H 9000 1850 50  0001 C CNN
 F 3 "" H 9000 1850 50  0001 C CNN
 	1    9000 1700
@@
 F 0 "H15" H 9200 1650 50  0000 R CNN
 F 1 "3V3" H 9200 1750 50  0000 R CNN
-F 2 "" H 9250 1850 50  0001 C CNN
+F 2 "Custom:Mounting_Pad_Power" H 9250 1850 50  0001 C CNN
 F 3 "" H 9250 1850 50  0001 C CNN
 	1    9250 1700
@@
 F 0 "H17" H 4500 7000 50  0000 R CNN
 F 1 "GND_TOUCH" H 4850 7100 50  0000 R CNN
-F 2 "" H 4350 7200 50  0001 C CNN
+F 2 "Custom:Mounting_Pad_Power" H 4350 7200 50  0001 C CNN
 F 3 "" H 4350 7200 50  0001 C CNN
 	1    4350 7050
@@
 F 0 "H16" H 4100 7000 50  0000 R CNN
 F 1 "GND_TOUCH" H 4100 7100 50  0000 R CNN
-F 2 "" H 4150 7200 50  0001 C CNN
+F 2 "Custom:Mounting_Pad_Power" H 4150 7200 50  0001 C CNN
 F 3 "" H 4150 7200 50  0001 C CNN
 	1    4150 7050

Commit message: Start renumber
Parts:
- M1, M2: footprint (none) -> Custom:K976_Stepper
Changed lines of the file:
@@
 F 0 "M1" H 5288 2874 50  0000 L CNN
 F 1 "Stepper_Motor_bipolar" H 5288 2783 50  0000 L CNN
-F 2 "" H 5110 2740 50  0001 C CNN
+F 2 "Custom:K976_Stepper" H 5110 2740 50  0001 C CNN
 F 3 "http://www.infineon.com/dgdl/Application-Note-TLE8110EE_driving_UniPolarStepperMotor_V1.1.pdf?fileId=db3a30431be39b97011be5d0aa0a00b0" H 5110 2740 50  0001 C CNN
 	1    5100 2750
@@
 F 0 "M2" H 5288 5474 50  0000 L CNN
 F 1 "Stepper_Motor_bipolar" H 5288 5383 50  0000 L CNN
-F 2 "" H 5110 5340 50  0001 C CNN
+F 2 "Custom:K976_Stepper" H 5110 5340 50  0001 C CNN
 F 3 "http://www.infineon.com/dgdl/Application-Note-TLE8110EE_driving_UniPolarStepperMotor_V1.1.pdf?fileId=db3a30431be39b97011be5d0aa0a00b0" H 5110 5340 50  0001 C CNN
 	1    5100 5350

Commit message: Finish bottom
Parts:
- added H18, H19: GND_TOUCH, Custom:Mounting_Pad_Ground, symbol Custom:MountingPad
- H16, H17: footprint Custom:Mounting_Pad_Power -> Custom:Mounting_Pad_Ground
Connections:
- net GND: now also H18.1 (Pin), H19.1 (Pin)
Other:
- moved on the sheet: H16, H17
Changed lines of the file:
@@
 L Custom:MountingPad H17
 U 1 1 5D91B15C
-P 4350 7050
-F 0 "H17" H 4500 7000 50  0000 R CNN
-F 1 "GND_TOUCH" H 4850 7100 50  0000 R CNN
-F 2 "Custom:Mounting_Pad_Power" H 4350 7200 50  0001 C CNN
-F 3 "" H 4350 7200 50  0001 C CNN
-	1    4350 7050
+P 3750 7050
+F 0 "H17" H 3950 7000 50  0000 R CNN
+F 1 "GND_TOUCH" H 4250 7100 50  0000 R CNN
+F 2 "Custom:Mounting_Pad_Ground" H 3750 7200 50  0001 C CNN
+F 3 "" H 3750 7200 50  0001 C CNN
+	1    3750 7050
 	1    0    0    -1
 $EndComp
@@
 L Custom:MountingPad H16
 U 1 1 5D91B695
-P 4150 7050
-F 0 "H16" H 4100 7000 50  0000 R CNN
-F 1 "GND_TOUCH" H 4100 7100 50  0000 R CNN
-F 2 "Custom:Mounting_Pad_Power" H 4150 7200 50  0001 C CNN
-F 3 "" H 4150 7200 50  0001 C CNN
-	1    4150 7050
+P 3550 7050
+F 0 "H16" H 3500 7000 50  0000 R CNN
+F 1 "GND_TOUCH" H 3500 7100 50  0000 R CNN
+F 2 "Custom:Mounting_Pad_Ground" H 3550 7200 50  0001 C CNN
+F 3 "" H 3550 7200 50  0001 C CNN
+	1    3550 7050
 	1    0    0    -1
 $EndComp
@@
 L power:GND #PWR011
 U 1 1 5D932EB6
-P 4150 7450
-F 0 "#PWR011" H 4150 7200 50  0001 C CNN
-F 1 "GND" H 4155 7277 50  0000 C CNN
-F 2 "" H 4150 7450 50  0001 C CNN
-F 3 "" H 4150 7450 50  0001 C CNN
-	1    4150 7450
+P 3550 7450
+F 0 "#PWR011" H 3550 7200 50  0001 C CNN
+F 1 "GND" H 3555 7277 50  0000 C CNN
+F 2 "" H 3550 7450 50  0001 C CNN
+F 3 "" H 3550 7450 50  0001 C CNN
+	1    3550 7450
 	1    0    0    -1
 $EndComp
@@
 L power:GND #PWR012
 U 1 1 5D9331C8
-P 4350 7450
-F 0 "#PWR012" H 4350 7200 50  0001 C CNN
-F 1 "GND" H 4355 7277 50  0000 C CNN
-F 2 "" H 4350 7450 50  0001 C CNN
-F 3 "" H 4350 7450 50  0001 C CNN
-	1    4350 7450
+P 3750 7450
+F 0 "#PWR012" H 3750 7200 50  0001 C CNN
+F 1 "GND" H 3755 7277 50  0000 C CNN
+F 2 "" H 3750 7450 50  0001 C CNN
+F 3 "" H 3750 7450 50  0001 C CNN
+	1    3750 7450
 	1    0    0    -1
 $EndComp
 Wire Wire Line
-	4150 7350 4150 7450
+	3550 7350 3550 7450
 $Comp
 L power:PWR_FLAG #FLG01
@@
 	10400 1050 10400 1150
 Wire Wire Line
-	4350 7350 4350 7450
+	3750 7350 3750 7450
 Text Notes 3800 6750 0    50   ~ 0
 PADS TO DRAG ON FLOOR
+$Comp
+L Custom:MountingPad H19
+U 1 1 5D86E5C3
+P 5000 7050
+F 0 "H19" H 5200 7000 50  0000 R CNN
+F 1 "GND_TOUCH" H 5500 7100 50  0000 R CNN
+F 2 "Custom:Mounting_Pad_Ground" H 5000 7200 50  0001 C CNN
+F 3 "" H 5000 7200 50  0001 C CNN
+	1    5000 7050
+	1    0    0    -1
+$EndComp
+$Comp
+L Custom:MountingPad H18
+U 1 1 5D86E5CD
+P 4800 7050
+F 0 "H18" H 4700 7000 50  0000 R CNN
+F 1 "GND_TOUCH" H 4750 7100 50  0000 R CNN
+F 2 "Custom:Mounting_Pad_Ground" H 4800 7200 50  0001 C CNN
+F 3 "" H 4800 7200 50  0001 C CNN
+	1    4800 7050
+	1    0    0    -1
+$EndComp
+$Comp
+L power:GND #PWR013
+U 1 1 5D86E5D7
+P 4800 7450
+F 0 "#PWR013" H 4800 7200 50  0001 C CNN
+F 1 "GND" H 4805 7277 50  0000 C CNN
+F 2 "" H 4800 7450 50  0001 C CNN
+F 3 "" H 4800 7450 50  0001 C CNN
+	1    4800 7450
+	1    0    0    -1
+$EndComp
+$Comp
+L power:GND #PWR014
+U 1 1 5D86E5E1
+P 5000 7450
+F 0 "#PWR014" H 5000 7200 50  0001 C CNN
+F 1 "GND" H 5005 7277 50  0000 C CNN
+F 2 "" H 5000 7450 50  0001 C CNN
+F 3 "" H 5000 7450 50  0001 C CNN
+	1    5000 7450
+	1    0    0    -1
+$EndComp
+Wire Wire Line
+	4800 7350 4800 7450
+Wire Wire Line
+	5000 7350 5000 7450
 $EndSCHEMATC

Commit message: Bottem changes
Parts:
- M1, M2: footprint Custom:K976_Stepper -> Custom:Medium_Stepper
Changed lines of the file:
@@
 F 0 "M1" H 5288 2874 50  0000 L CNN
 F 1 "Stepper_Motor_bipolar" H 5288 2783 50  0000 L CNN
-F 2 "Custom:K976_Stepper" H 5110 2740 50  0001 C CNN
+F 2 "Custom:Medium_Stepper" H 5110 2740 50  0001 C CNN
 F 3 "http://www.infineon.com/dgdl/Application-Note-TLE8110EE_driving_UniPolarStepperMotor_V1.1.pdf?fileId=db3a30431be39b97011be5d0aa0a00b0" H 5110 2740 50  0001 C CNN
 	1    5100 2750
@@
 F 0 "M2" H 5288 5474 50  0000 L CNN
 F 1 "Stepper_Motor_bipolar" H 5288 5383 50  0000 L CNN
-F 2 "Custom:K976_Stepper" H 5110 5340 50  0001 C CNN
+F 2 "Custom:Medium_Stepper" H 5110 5340 50  0001 C CNN
 F 3 "http://www.infineon.com/dgdl/Application-Note-TLE8110EE_driving_UniPolarStepperMotor_V1.1.pdf?fileId=db3a30431be39b97011be5d0aa0a00b0" H 5110 5340 50  0001 C CNN
 	1    5100 5350

Commit message: Finisch bottom
Parts:
- C10, C11, C12, C13, C8, C9: footprint Capacitors_SMD:C_1206 -> Capacitors_SMD:C_0805
- R1, R11, R12, R13, R14, R2, R3, R4: footprint Resistors_SMD:R_1206 -> Resistors_SMD:R_0805
Changed lines of the file:
@@
 F 0 "C9" H 3015 1696 50  0000 L CNN
 F 1 "2.2µ" H 3015 1605 50  0000 L CNN
-F 2 "Capacitors_SMD:C_1206" H 2938 1500 50  0001 C CNN
+F 2 "Capacitors_SMD:C_0805" H 2938 1500 50  0001 C CNN
 F 3 "~" H 2900 1650 50  0001 C CNN
 	1    2900 1650
@@
 F 0 "C8" H 1865 1696 50  0000 L CNN
 F 1 "0.01µ" H 1865 1605 50  0000 L CNN
-F 2 "Capacitors_SMD:C_1206" H 1788 1500 50  0001 C CNN
+F 2 "Capacitors_SMD:C_0805" H 1788 1500 50  0001 C CNN
 F 3 "~" H 1750 1650 50  0001 C CNN
 	1    1750 1650
@@
 F 0 "C10" H 3815 1696 50  0000 L CNN
 F 1 "10µ" H 3815 1605 50  0000 L CNN
-F 2 "Capacitors_SMD:C_1206" H 3738 1500 50  0001 C CNN
+F 2 "Capacitors_SMD:C_0805" H 3738 1500 50  0001 C CNN
 F 3 "~" H 3700 1650 50  0001 C CNN
 	1    3700 1650
@@
 F 0 "R11" H 1370 2796 50  0000 L CNN
 F 1 "0.8" H 1370 2705 50  0000 L CNN
-F 2 "Resistors_SMD:R_1206" V 1230 2750 50  0001 C CNN
+F 2 "Resistors_SMD:R_0805" V 1230 2750 50  0001 C CNN
 F 3 "~" H 1300 2750 50  0001 C CNN
 	1    1300 2750
@@
 F 0 "R12" H 1720 2796 50  0000 L CNN
 F 1 "0.8" H 1720 2705 50  0000 L CNN
-F 2 "Resistors_SMD:R_1206" V 1580 2750 50  0001 C CNN
+F 2 "Resistors_SMD:R_0805" V 1580 2750 50  0001 C CNN
 F 3 "~" H 1650 2750 50  0001 C CNN
 	1    1650 2750
@@
 F 0 "C12" H 3015 4296 50  0000 L CNN
 F 1 "2.2µ" H 3015 4205 50  0000 L CNN
-F 2 "Capacitors_SMD:C_1206" H 2938 4100 50  0001 C CNN
+F 2 "Capacitors_SMD:C_0805" H 2938 4100 50  0001 C CNN
 F 3 "~" H 2900 4250 50  0001 C CNN
 	1    2900 4250
@@
 F 0 "C11" H 1865 4296 50  0000 L CNN
 F 1 "0.01µ" H 1865 4205 50  0000 L CNN
-F 2 "Capacitors_SMD:C_1206" H 1788 4100 50  0001 C CNN
+F 2 "Capacitors_SMD:C_0805" H 1788 4100 50  0001 C CNN
 F 3 "~" H 1750 4250 50  0001 C CNN
 	1    1750 4250
@@
 F 0 "C13" H 3815 4296 50  0000 L CNN
 F 1 "10µ" H 3815 4205 50  0000 L CNN
-F 2 "Capacitors_SMD:C_1206" H 3738 4100 50  0001 C CNN
+F 2 "Capacitors_SMD:C_0805" H 3738 4100 50  0001 C CNN
 F 3 "~" H 3700 4250 50  0001 C CNN
 	1    3700 4250
@@
 F 0 "R13" H 1370 5396 50  0000 L CNN
 F 1 "0.8" H 1370 5305 50  0000 L CNN
-F 2 "Resistors_SMD:R_1206" V 1230 5350 50  0001 C CNN
+F 2 "Resistors_SMD:R_0805" V 1230 5350 50  0001 C CNN
 F 3 "~" H 1300 5350 50  0001 C CNN
 	1    1300 5350
@@
 F 0 "R14" H 1720 5396 50  0000 L CNN
 F 1 "0.8" H 1720 5305 50  0000 L CNN
-F 2 "Resistors_SMD:R_1206" V 1580 5350 50  0001 C CNN
+F 2 "Resistors_SMD:R_0805" V 1580 5350 50  0001 C CNN
 F 3 "~" H 1650 5350 50  0001 C CNN
 	1    1650 5350
@@
 F 0 "R2" H 8020 3346 50  0000 L CNN
 F 1 "120" H 8020 3255 50  0000 L CNN
-F 2 "Resistors_SMD:R_1206" V 7880 3300 50  0001 C CNN
+F 2 "Resistors_SMD:R_0805" V 7880 3300 50  0001 C CNN
 F 3 "~" H 7950 3300 50  0001 C CNN
 	1    7950 3300
@@
 F 0 "R1" H 7620 3346 50  0000 L CNN
 F 1 "10k" H 7620 3255 50  0000 L CNN
-F 2 "Resistors_SMD:R_1206" V 7480 3300 50  0001 C CNN
+F 2 "Resistors_SMD:R_0805" V 7480 3300 50  0001 C CNN
 F 3 "~" H 7550 3300 50  0001 C CNN
 	1    7550 3300
@@
 F 0 "R4" H 9820 3346 50  0000 L CNN
 F 1 "120" H 9820 3255 50  0000 L CNN
-F 2 "Resistors_SMD:R_1206" V 9680 3300 50  0001 C CNN
+F 2 "Resistors_SMD:R_0805" V 9680 3300 50  0001 C CNN
 F 3 "~" H 9750 3300 50  0001 C CNN
 	1    9750 3300
@@
 F 0 "R3" H 9420 3346 50  0000 L CNN
 F 1 "10k" H 9420 3255 50  0000 L CNN
-F 2 "Resistors_SMD:R_1206" V 9280 3300 50  0001 C CNN
+F 2 "Resistors_SMD:R_0805" V 9280 3300 50  0001 C CNN
 F 3 "~" H 9350 3300 50  0001 C CNN
 	1    9350 3300
