File: robot/Bottom/Bottom.sch (KiCad schematic (older format))
At the start: 39 parts, among them M1 Stepper_Motor_bipolar, M2 Stepper_Motor_bipolar, U1 GP2S60, U2 GP2S60, U7 DRV8833PWP, U8 DRV8833PWP

Commit message: Changes to structure
Parts:
- added J1, J4, J5: Conn_01x02, Connector_PinSocket_2.54mm:PinSocket_1x02_P2.54mm_Horizontal, symbol Connector_Generic:Conn_01x02
- added J2, J3: Conn_01x01, Connector_PinSocket_2.54mm:PinSocket_1x01_P2.54mm_Horizontal, symbol Connector_Generic:Conn_01x01
Connections:
- no-connect marks 2 -> 10
Other:
- note added: "Assembly"
Changed lines of the file:
@@
 EESchema Schematic File Version 4
 LIBS:Bottom-cache
-EELAYER 29 0
+EELAYER 30 0
 EELAYER END
 $Descr A4 11693 8268
@@
 Wire Wire Line
 	5000 7350 5000 7450
+NoConn ~ 9150 5150
+NoConn ~ 9050 5150
+NoConn ~ 8750 5150
+NoConn ~ 8650 5150
+NoConn ~ 8350 5150
+NoConn ~ 8250 5150
+NoConn ~ 8350 6000
+NoConn ~ 8350 5750
+$Comp
+L Connector_Generic:Conn_01x01 J3
+U 1 1 5D93F861
+P 8550 6000
+F 0 "J3" H 8630 6042 50  0000 L CNN
+F 1 "Conn_01x01" H 8630 5951 50  0000 L CNN
+F 2 "Connector_PinSocket_2.54mm:PinSocket_1x01_P2.54mm_Horizontal" H 8550 6000 50  0001 C CNN
+F 3 "~" H 8550 6000 50  0001 C CNN
+	1    8550 6000
+	1    0    0    -1
+$EndComp
+$Comp
+L Connector_Generic:Conn_01x01 J2
+U 1 1 5D93EA93
+P 8550 5750
+F 0 "J2" H 8630 5792 50  0000 L CNN
+F 1 "Conn_01x01" H 8630 5701 50  0000 L CNN
+F 2 "Connector_PinSocket_2.54mm:PinSocket_1x01_P2.54mm_Horizontal" H 8550 5750 50  0001 C CNN
+F 3 "~" H 8550 5750 50  0001 C CNN
+	1    8550 5750
+	1    0    0    -1
+$EndComp
+$Comp
+L Connector_Generic:Conn_01x02 J5
+U 1 1 5D93E328
+P 9150 5350
+F 0 "J5" V 9022 5430 50  0000 L CNN
+F 1 "Conn_01x02" V 9250 5100 50  0000 L CNN
+F 2 "Connector_PinSocket_2.54mm:PinSocket_1x02_P2.54mm_Horizontal" H 9150 5350 50  0001 C CNN
+F 3 "~" H 9150 5350 50  0001 C CNN
+	1    9150 5350
+	0    1    1    0
+$EndComp
+$Comp
+L Connector_Generic:Conn_01x02 J4
+U 1 1 5D93DC92
+P 8750 5350
+F 0 "J4" V 8622 5430 50  0000 L CNN
+F 1 "Conn_01x02" V 8950 5100 50  0000 L CNN
+F 2 "Connector_PinSocket_2.54mm:PinSocket_1x02_P2.54mm_Horizontal" H 8750 5350 50  0001 C CNN
+F 3 "~" H 8750 5350 50  0001 C CNN
+	1    8750 5350
+	0    1    1    0
+$EndComp
+$Comp
+L Connector_Generic:Conn_01x02 J1
+U 1 1 5D9381E5
+P 8350 5350
+F 0 "J1" V 8222 5430 50  0000 L CNN
+F 1 "Conn_01x02" V 8450 5100 50  0000 L CNN
+F 2 "Connector_PinSocket_2.54mm:PinSocket_1x02_P2.54mm_Horizontal" H 8350 5350 50  0001 C CNN
+F 3 "~" H 8350 5350 50  0001 C CNN
+	1    8350 5350
+	0    1    1    0
+$EndComp
+Text Notes 8550 5000 0    50   ~ 0
+Assembly
 $EndSCHEMATC

Commit message: Top changes
Parts:
- removed J1, J5: Conn_01x02, Connector_PinSocket_2.54mm:PinSocket_1x02_P2.54mm_Horizontal, symbol Connector_Generic:Conn_01x02
- added J? (x2): Conn_01x01, Connector_PinSocket_2.54mm:PinSocket_1x01_P2.54mm_Horizontal, symbol Connector_Generic:Conn_01x01
Connections:
- no-connect marks 10 -> 8
Other:
- moved on the sheet: J2, J3
Changed lines of the file:
@@
 Wire Wire Line
 	5000 7350 5000 7450
-NoConn ~ 9150 5150
-NoConn ~ 9050 5150
 NoConn ~ 8750 5150
 NoConn ~ 8650 5150
-NoConn ~ 8350 5150
-NoConn ~ 8250 5150
-NoConn ~ 8350 6000
-NoConn ~ 8350 5750
+NoConn ~ 8100 6000
+NoConn ~ 8100 5750
 $Comp
 L Connector_Generic:Conn_01x01 J3
 U 1 1 5D93F861
-P 8550 6000
-F 0 "J3" H 8630 6042 50  0000 L CNN
-F 1 "Conn_01x01" H 8630 5951 50  0000 L CNN
-F 2 "Connector_PinSocket_2.54mm:PinSocket_1x01_P2.54mm_Horizontal" H 8550 6000 50  0001 C CNN
-F 3 "~" H 8550 6000 50  0001 C CNN
-	1    8550 6000
+P 8300 6000
+F 0 "J3" H 8380 6042 50  0000 L CNN
+F 1 "Conn_01x01" H 8380 5951 50  0000 L CNN
+F 2 "Connector_PinSocket_2.54mm:PinSocket_1x01_P2.54mm_Horizontal" H 8300 6000 50  0001 C CNN
+F 3 "~" H 8300 6000 50  0001 C CNN
+	1    8300 6000
 	1    0    0    -1
 $EndComp
@@
 L Connector_Generic:Conn_01x01 J2
 U 1 1 5D93EA93
-P 8550 5750
-F 0 "J2" H 8630 5792 50  0000 L CNN
-F 1 "Conn_01x01" H 8630 5701 50  0000 L CNN
-F 2 "Connector_PinSocket_2.54mm:PinSocket_1x01_P2.54mm_Horizontal" H 8550 5750 50  0001 C CNN
-F 3 "~" H 8550 5750 50  0001 C CNN
-	1    8550 5750
+P 8300 5750
+F 0 "J2" H 8380 5792 50  0000 L CNN
+F 1 "Conn_01x01" H 8380 5701 50  0000 L CNN
+F 2 "Connector_PinSocket_2.54mm:PinSocket_1x01_P2.54mm_Horizontal" H 8300 5750 50  0001 C CNN
+F 3 "~" H 8300 5750 50  0001 C CNN
+	1    8300 5750
 	1    0    0    -1
-$EndComp
-$Comp
-L Connector_Generic:Conn_01x02 J5
-U 1 1 5D93E328
-P 9150 5350
-F 0 "J5" V 9022 5430 50  0000 L CNN
-F 1 "Conn_01x02" V 9250 5100 50  0000 L CNN
-F 2 "Connector_PinSocket_2.54mm:PinSocket_1x02_P2.54mm_Horizontal" H 9150 5350 50  0001 C CNN
-F 3 "~" H 9150 5350 50  0001 C CNN
-	1    9150 5350
-	0    1    1    0
 $EndComp
 $Comp
@@
 	0    1    1    0
 $EndComp
-$Comp
-L Connector_Generic:Conn_01x02 J1
-U 1 1 5D9381E5
-P 8350 5350
-F 0 "J1" V 8222 5430 50  0000 L CNN
-F 1 "Conn_01x02" V 8450 5100 50  0000 L CNN
-F 2 "Connector_PinSocket_2.54mm:PinSocket_1x02_P2.54mm_Horizontal" H 8350 5350 50  0001 C CNN
-F 3 "~" H 8350 5350 50  0001 C CNN
-	1    8350 5350
-	0    1    1    0
-$EndComp
 Text Notes 8550 5000 0    50   ~ 0
 Assembly
+NoConn ~ 8950 6000
+NoConn ~ 8950 5750
+$Comp
+L Connector_Generic:Conn_01x01 J?
+U 1 1 5D950907
+P 9150 6000
+F 0 "J?" H 9230 6042 50  0000 L CNN
+F 1 "Conn_01x01" H 9230 5951 50  0000 L CNN
+F 2 "Connector_PinSocket_2.54mm:PinSocket_1x01_P2.54mm_Horizontal" H 9150 6000 50  0001 C CNN
+F 3 "~" H 9150 6000 50  0001 C CNN
+	1    9150 6000
+	1    0    0    -1
+$EndComp
+$Comp
+L Connector_Generic:Conn_01x01 J?
+U 1 1 5D95090D
+P 9150 5750
+F 0 "J?" H 9230 5792 50  0000 L CNN
+F 1 "Conn_01x01" H 9230 5701 50  0000 L CNN
+F 2 "Connector_PinSocket_2.54mm:PinSocket_1x01_P2.54mm_Horizontal" H 9150 5750 50  0001 C CNN
+F 3 "~" H 9150 5750 50  0001 C CNN
+	1    9150 5750
+	1    0    0    -1
+$EndComp
 $EndSCHEMATC
