File: robot/Bottom/Bottom.sch (KiCad schematic (older format))
At the start: 44 parts, among them J2 Conn_01x01, J3 Conn_01x01, J4 Conn_01x02, M1 Stepper_Motor_bipolar, M2 Stepper_Motor_bipolar, U1 GP2S60, U2 GP2S60, U7 DRV8833PWP, U8 DRV8833PWP

Commit message: Small changes, connectors
Parts:
- removed J2, J3, J? (x2): Conn_01x01, Connector_PinSocket_2.54mm:PinSocket_1x01_P2.54mm_Horizontal, symbol Connector_Generic:Conn_01x01
- removed J4: Conn_01x02, Connector_PinSocket_2.54mm:PinSocket_1x02_P2.54mm_Horizontal, symbol Connector_Generic:Conn_01x02
- added H20, H21: GND, Custom:Mounting_Pad_Power, symbol Custom:MountingPad
- added J1: Conn_01x02, Custom:BG300-02-A-L-A, symbol Connector_Generic:Conn_01x02
- C10, C11, C12, C13, C8, C9: footprint Capacitors_SMD:C_0805 -> Capacitor_SMD:C_0805_2012Metric
- R1, R11, R12, R13, R14, R2, R3, R4: footprint Resistors_SMD:R_0805 -> Resistor_SMD:R_0805_2012Metric
Connections:
- net GND: now also H20.1 (Pin), H21.1 (Pin)
- no-connect marks 8 -> 4
Changed lines of the file:
@@
 F 0 "C9" H 3015 1696 50  0000 L CNN
 F 1 "2.2µ" H 3015 1605 50  0000 L CNN
-F 2 "Capacitors_SMD:C_0805" H 2938 1500 50  0001 C CNN
+F 2 "Capacitor_SMD:C_0805_2012Metric" H 2938 1500 50  0001 C CNN
 F 3 "~" H 2900 1650 50  0001 C CNN
 	1    2900 1650
@@
 F 0 "C8" H 1865 1696 50  0000 L CNN
 F 1 "0.01µ" H 1865 1605 50  0000 L CNN
-F 2 "Capacitors_SMD:C_0805" H 1788 1500 50  0001 C CNN
+F 2 "Capacitor_SMD:C_0805_2012Metric" H 1788 1500 50  0001 C CNN
 F 3 "~" H 1750 1650 50  0001 C CNN
 	1    1750 1650
@@
 F 0 "C10" H 3815 1696 50  0000 L CNN
 F 1 "10µ" H 3815 1605 50  0000 L CNN
-F 2 "Capacitors_SMD:C_0805" H 3738 1500 50  0001 C CNN
+F 2 "Capacitor_SMD:C_0805_2012Metric" H 3738 1500 50  0001 C CNN
 F 3 "~" H 3700 1650 50  0001 C CNN
 	1    3700 1650
@@
 F 0 "R11" H 1370 2796 50  0000 L CNN
 F 1 "0.8" H 1370 2705 50  0000 L CNN
-F 2 "Resistors_SMD:R_0805" V 1230 2750 50  0001 C CNN
+F 2 "Resistor_SMD:R_0805_2012Metric" V 1230 2750 50  0001 C CNN
 F 3 "~" H 1300 2750 50  0001 C CNN
 	1    1300 2750
@@
 F 0 "R12" H 1720 2796 50  0000 L CNN
 F 1 "0.8" H 1720 2705 50  0000 L CNN
-F 2 "Resistors_SMD:R_0805" V 1580 2750 50  0001 C CNN
+F 2 "Resistor_SMD:R_0805_2012Metric" V 1580 2750 50  0001 C CNN
 F 3 "~" H 1650 2750 50  0001 C CNN
 	1    1650 2750
@@
 F 0 "C12" H 3015 4296 50  0000 L CNN
 F 1 "2.2µ" H 3015 4205 50  0000 L CNN
-F 2 "Capacitors_SMD:C_0805" H 2938 4100 50  0001 C CNN
+F 2 "Capacitor_SMD:C_0805_2012Metric" H 2938 4100 50  0001 C CNN
 F 3 "~" H 2900 4250 50  0001 C CNN
 	1    2900 4250
@@
 F 0 "C11" H 1865 4296 50  0000 L CNN
 F 1 "0.01µ" H 1865 4205 50  0000 L CNN
-F 2 "Capacitors_SMD:C_0805" H 1788 4100 50  0001 C CNN
+F 2 "Capacitor_SMD:C_0805_2012Metric" H 1788 4100 50  0001 C CNN
 F 3 "~" H 1750 4250 50  0001 C CNN
 	1    1750 4250
@@
 F 0 "C13" H 3815 4296 50  0000 L CNN
 F 1 "10µ" H 3815 4205 50  0000 L CNN
-F 2 "Capacitors_SMD:C_0805" H 3738 4100 50  0001 C CNN
+F 2 "Capacitor_SMD:C_0805_2012Metric" H 3738 4100 50  0001 C CNN
 F 3 "~" H 3700 4250 50  0001 C CNN
 	1    3700 4250
@@
 F 0 "R13" H 1370 5396 50  0000 L CNN
 F 1 "0.8" H 1370 5305 50  0000 L CNN
-F 2 "Resistors_SMD:R_0805" V 1230 5350 50  0001 C CNN
+F 2 "Resistor_SMD:R_0805_2012Metric" V 1230 5350 50  0001 C CNN
 F 3 "~" H 1300 5350 50  0001 C CNN
 	1    1300 5350
@@
 F 0 "R14" H 1720 5396 50  0000 L CNN
 F 1 "0.8" H 1720 5305 50  0000 L CNN
-F 2 "Resistors_SMD:R_0805" V 1580 5350 50  0001 C CNN
+F 2 "Resistor_SMD:R_0805_2012Metric" V 1580 5350 50  0001 C CNN
 F 3 "~" H 1650 5350 50  0001 C CNN
 	1    1650 5350
@@
 F 0 "R2" H 8020 3346 50  0000 L CNN
 F 1 "120" H 8020 3255 50  0000 L CNN
-F 2 "Resistors_SMD:R_0805" V 7880 3300 50  0001 C CNN
+F 2 "Resistor_SMD:R_0805_2012Metric" V 7880 3300 50  0001 C CNN
 F 3 "~" H 7950 3300 50  0001 C CNN
 	1    7950 3300
@@
 F 0 "R1" H 7620 3346 50  0000 L CNN
 F 1 "10k" H 7620 3255 50  0000 L CNN
-F 2 "Resistors_SMD:R_0805" V 7480 3300 50  0001 C CNN
+F 2 "Resistor_SMD:R_0805_2012Metric" V 7480 3300 50  0001 C CNN
 F 3 "~" H 7550 3300 50  0001 C CNN
 	1    7550 3300
@@
 F 0 "R4" H 9820 3346 50  0000 L CNN
 F 1 "120" H 9820 3255 50  0000 L CNN
-F 2 "Resistors_SMD:R_0805" V 9680 3300 50  0001 C CNN
+F 2 "Resistor_SMD:R_0805_2012Metric" V 9680 3300 50  0001 C CNN
 F 3 "~" H 9750 3300 50  0001 C CNN
 	1    9750 3300
@@
 F 0 "R3" H 9420 3346 50  0000 L CNN
 F 1 "10k" H 9420 3255 50  0000 L CNN
-F 2 "Resistors_SMD:R_0805" V 9280 3300 50  0001 C CNN
+F 2 "Resistor_SMD:R_0805_2012Metric" V 9280 3300 50  0001 C CNN
 F 3 "~" H 9350 3300 50  0001 C CNN
 	1    9350 3300
@@
 Wire Wire Line
 	5000 7350 5000 7450
-NoConn ~ 8750 5150
-NoConn ~ 8650 5150
-NoConn ~ 8100 6000
-NoConn ~ 8100 5750
-$Comp
-L Connector_Generic:Conn_01x01 J3
-U 1 1 5D93F861
-P 8300 6000
-F 0 "J3" H 8380 6042 50  0000 L CNN
-F 1 "Conn_01x01" H 8380 5951 50  0000 L CNN
-F 2 "Connector_PinSocket_2.54mm:PinSocket_1x01_P2.54mm_Horizontal" H 8300 6000 50  0001 C CNN
-F 3 "~" H 8300 6000 50  0001 C CNN
-	1    8300 6000
-	1    0    0    -1
-$EndComp
-$Comp
-L Connector_Generic:Conn_01x01 J2
-U 1 1 5D93EA93
-P 8300 5750
-F 0 "J2" H 8380 5792 50  0000 L CNN
-F 1 "Conn_01x01" H 8380 5701 50  0000 L CNN
-F 2 "Connector_PinSocket_2.54mm:PinSocket_1x01_P2.54mm_Horizontal" H 8300 5750 50  0001 C CNN
-F 3 "~" H 8300 5750 50  0001 C CNN
-	1    8300 5750
-	1    0    0    -1
-$EndComp
-$Comp
-L Connector_Generic:Conn_01x02 J4
-U 1 1 5D93DC92
-P 8750 5350
-F 0 "J4" V 8622 5430 50  0000 L CNN
-F 1 "Conn_01x02" V 8950 5100 50  0000 L CNN
-F 2 "Connector_PinSocket_2.54mm:PinSocket_1x02_P2.54mm_Horizontal" H 8750 5350 50  0001 C CNN
-F 3 "~" H 8750 5350 50  0001 C CNN
-	1    8750 5350
-	0    1    1    0
-$EndComp
 Text Notes 8550 5000 0    50   ~ 0
 Assembly
-NoConn ~ 8950 6000
-NoConn ~ 8950 5750
-$Comp
-L Connector_Generic:Conn_01x01 J?
-U 1 1 5D950907
-P 9150 6000
-F 0 "J?" H 9230 6042 50  0000 L CNN
-F 1 "Conn_01x01" H 9230 5951 50  0000 L CNN
-F 2 "Connector_PinSocket_2.54mm:PinSocket_1x01_P2.54mm_Horizontal" H 9150 6000 50  0001 C CNN
-F 3 "~" H 9150 6000 50  0001 C CNN
-	1    9150 6000
-	1    0    0    -1
-$EndComp
-$Comp
-L Connector_Generic:Conn_01x01 J?
-U 1 1 5D95090D
-P 9150 5750
-F 0 "J?" H 9230 5792 50  0000 L CNN
-F 1 "Conn_01x01" H 9230 5701 50  0000 L CNN
-F 2 "Connector_PinSocket_2.54mm:PinSocket_1x01_P2.54mm_Horizontal" H 9150 5750 50  0001 C CNN
-F 3 "~" H 9150 5750 50  0001 C CNN
-	1    9150 5750
-	1    0    0    -1
-$EndComp
+$Comp
+L Custom:MountingPad H20
+U 1 1 5D98F825
+P 7850 1700
+F 0 "H20" H 7750 1750 50  0000 R CNN
+F 1 "GND" H 7750 1650 50  0000 R CNN
+F 2 "Custom:Mounting_Pad_Power" H 7850 1850 50  0001 C CNN
+F 3 "" H 7850 1850 50  0001 C CNN
+	1    7850 1700
+	1    0    0    -1
+$EndComp
+$Comp
+L power:GND #PWR0101
+U 1 1 5D98F82F
+P 7850 2100
+F 0 "#PWR0101" H 7850 1850 50  0001 C CNN
+F 1 "GND" H 7855 1927 50  0000 C CNN
+F 2 "" H 7850 2100 50  0001 C CNN
+F 3 "" H 7850 2100 50  0001 C CNN
+	1    7850 2100
+	1    0    0    -1
+$EndComp
+Wire Wire Line
+	7850 2000 7850 2100
+$Comp
+L Custom:MountingPad H21
+U 1 1 5D9A8D04
+P 9500 1700
+F 0 "H21" H 9650 1750 50  0000 R CNN
+F 1 "GND" H 9700 1650 50  0000 R CNN
+F 2 "Custom:Mounting_Pad_Power" H 9500 1850 50  0001 C CNN
+F 3 "" H 9500 1850 50  0001 C CNN
+	1    9500 1700
+	1    0    0    -1
+$EndComp
+$Comp
+L power:GND #PWR0102
+U 1 1 5D9A8D0E
+P 9500 2100
+F 0 "#PWR0102" H 9500 1850 50  0001 C CNN
+F 1 "GND" H 9505 1927 50  0000 C CNN
+F 2 "" H 9500 2100 50  0001 C CNN
+F 3 "" H 9500 2100 50  0001 C CNN
+	1    9500 2100
+	1    0    0    -1
+$EndComp
+Wire Wire Line
+	9500 2000 9500 2100
+$Comp
+L Connector_Generic:Conn_01x02 J1
+U 1 1 5D98AE31
+P 8750 5450
+F 0 "J1" V 8622 5530 50  0000 L CNN
+F 1 "Conn_01x02" V 8713 5530 50  0000 L CNN
+F 2 "Custom:BG300-02-A-L-A" H 8750 5450 50  0001 C CNN
+F 3 "~" H 8750 5450 50  0001 C CNN
+	1    8750 5450
+	0    1    1    0
+$EndComp
+NoConn ~ 8750 5250
+NoConn ~ 8650 5250
 $EndSCHEMATC

Commit message: BOM items
Parts:
- removed J1: Conn_01x02, Custom:BG300-02-A-L-A, symbol Connector_Generic:Conn_01x02
- C10, C13: value 10µ -> 22µ; LCSC (none) -> C5674; Manufacturer Nbr (none) -> CL21A226MQQNNNE
- C11, C8: LCSC (none) -> C52278; Manufacturer Nbr (none) -> 0805B103K500NT
- C12, C9: LCSC (none) -> C107171; Manufacturer Nbr (none) -> CC0805ZRY5V7BB225
- H11: value M_~SLP -> M~SLP
- R1, R3: LCSC (none) -> C38522; Manufacturer Nbr (none) -> 0805W8F1002T5E
- R11, R12, R13, R14: value 0.8 -> 1; LCSC (none) -> C25288; Manufacturer Nbr (none) -> 0805W8J010JT5E
- R2, R4: LCSC (none) -> C25281; Manufacturer Nbr (none) -> 0805W8J0120T5E
- U1, U2: LCSC (none) -> C83485; Manufacturer Nbr (none) -> GP2S60B
- U7, U8: Farnell (none) -> 2057085RL
Connections:
- no-connect marks 4 -> 2
Other:
- note removed: "Assembly"
Changed lines of the file:
@@
 F 2 "Package_SO:HTSSOP-16-1EP_4.4x5mm_P0.65mm_EP3.4x5mm_Mask2.46x2.31mm_ThermalVias" H 3450 3050 50  0001 L CNN
 F 3 "http://www.ti.com/lit/ds/symlink/drv8833.pdf" H 2850 3150 50  0001 C CNN
+F 4 "2057085RL" H 3000 2600 50  0001 C CNN "Farnell"
 	1    3000 2600
 	1    0    0    -1
@@
 F 2 "Capacitor_SMD:C_0805_2012Metric" H 2938 1500 50  0001 C CNN
 F 3 "~" H 2900 1650 50  0001 C CNN
+F 4 "C107171" H 2900 1650 50  0001 C CNN "LCSC"
+F 5 "CC0805ZRY5V7BB225" H 2900 1650 50  0001 C CNN "Manufacturer Nbr"
 	1    2900 1650
 	1    0    0    -1
@@
 F 2 "Capacitor_SMD:C_0805_2012Metric" H 1788 1500 50  0001 C CNN
 F 3 "~" H 1750 1650 50  0001 C CNN
+F 4 "C52278" H 1750 1650 50  0001 C CNN "LCSC"
+F 5 "0805B103K500NT" H 1750 1650 50  0001 C CNN "Manufacturer Nbr"
 	1    1750 1650
 	1    0    0    -1
@@
 P 3700 1650
 F 0 "C10" H 3815 1696 50  0000 L CNN
-F 1 "10µ" H 3815 1605 50  0000 L CNN
+F 1 "22µ" H 3815 1605 50  0000 L CNN
 F 2 "Capacitor_SMD:C_0805_2012Metric" H 3738 1500 50  0001 C CNN
 F 3 "~" H 3700 1650 50  0001 C CNN
+F 4 "C5674" H 3700 1650 50  0001 C CNN "LCSC"
+F 5 "CL21A226MQQNNNE" H 3700 1650 50  0001 C CNN "Manufacturer Nbr"
 	1    3700 1650
 	1    0    0    -1
@@
 P 1300 2750
 F 0 "R11" H 1370 2796 50  0000 L CNN
-F 1 "0.8" H 1370 2705 50  0000 L CNN
+F 1 "1" H 1370 2705 50  0000 L CNN
 F 2 "Resistor_SMD:R_0805_2012Metric" V 1230 2750 50  0001 C CNN
 F 3 "~" H 1300 2750 50  0001 C CNN
+F 4 "C25288" H 1300 2750 50  0001 C CNN "LCSC"
+F 5 "0805W8J010JT5E" H 1300 2750 50  0001 C CNN "Manufacturer Nbr"
 	1    1300 2750
 	1    0    0    -1
@@
 P 1650 2750
 F 0 "R12" H 1720 2796 50  0000 L CNN
-F 1 "0.8" H 1720 2705 50  0000 L CNN
+F 1 "1" H 1720 2705 50  0000 L CNN
 F 2 "Resistor_SMD:R_0805_2012Metric" V 1580 2750 50  0001 C CNN
 F 3 "~" H 1650 2750 50  0001 C CNN
+F 4 "C25288" H 1650 2750 50  0001 C CNN "LCSC"
+F 5 "0805W8J010JT5E" H 1650 2750 50  0001 C CNN "Manufacturer Nbr"
 	1    1650 2750
 	1    0    0    -1
@@
 F 2 "Package_SO:HTSSOP-16-1EP_4.4x5mm_P0.65mm_EP3.4x5mm_Mask2.46x2.31mm_ThermalVias" H 3450 5650 50  0001 L CNN
 F 3 "http://www.ti.com/lit/ds/symlink/drv8833.pdf" H 2850 5750 50  0001 C CNN
+F 4 "2057085RL" H 3000 5200 50  0001 C CNN "Farnell"
 	1    3000 5200
 	1    0    0    -1
@@
 F 2 "Capacitor_SMD:C_0805_2012Metric" H 2938 4100 50  0001 C CNN
 F 3 "~" H 2900 4250 50  0001 C CNN
+F 4 "C107171" H 2900 4250 50  0001 C CNN "LCSC"
+F 5 "CC0805ZRY5V7BB225" H 2900 4250 50  0001 C CNN "Manufacturer Nbr"
 	1    2900 4250
 	1    0    0    -1
@@
 F 2 "Capacitor_SMD:C_0805_2012Metric" H 1788 4100 50  0001 C CNN
 F 3 "~" H 1750 4250 50  0001 C CNN
+F 4 "C52278" H 1750 4250 50  0001 C CNN "LCSC"
+F 5 "0805B103K500NT" H 1750 4250 50  0001 C CNN "Manufacturer Nbr"
 	1    1750 4250
 	1    0    0    -1
@@
 P 3700 4250
 F 0 "C13" H 3815 4296 50  0000 L CNN
-F 1 "10µ" H 3815 4205 50  0000 L CNN
+F 1 "22µ" H 3815 4205 50  0000 L CNN
 F 2 "Capacitor_SMD:C_0805_2012Metric" H 3738 4100 50  0001 C CNN
 F 3 "~" H 3700 4250 50  0001 C CNN
+F 4 "C5674" H 3700 4250 50  0001 C CNN "LCSC"
+F 5 "CL21A226MQQNNNE" H 3700 4250 50  0001 C CNN "Manufacturer Nbr"
 	1    3700 4250
 	1    0    0    -1
@@
 P 1300 5350
 F 0 "R13" H 1370 5396 50  0000 L CNN
-F 1 "0.8" H 1370 5305 50  0000 L CNN
+F 1 "1" H 1370 5305 50  0000 L CNN
 F 2 "Resistor_SMD:R_0805_2012Metric" V 1230 5350 50  0001 C CNN
 F 3 "~" H 1300 5350 50  0001 C CNN
+F 4 "C25288" H 1300 5350 50  0001 C CNN "LCSC"
+F 5 "0805W8J010JT5E" H 1300 5350 50  0001 C CNN "Manufacturer Nbr"
 	1    1300 5350
 	1    0    0    -1
@@
 P 1650 5350
 F 0 "R14" H 1720 5396 50  0000 L CNN
-F 1 "0.8" H 1720 5305 50  0000 L CNN
+F 1 "1" H 1720 5305 50  0000 L CNN
 F 2 "Resistor_SMD:R_0805_2012Metric" V 1580 5350 50  0001 C CNN
 F 3 "~" H 1650 5350 50  0001 C CNN
+F 4 "C25288" H 1650 5350 50  0001 C CNN "LCSC"
+F 5 "0805W8J010JT5E" H 1650 5350 50  0001 C CNN "Manufacturer Nbr"
 	1    1650 5350
 	1    0    0    -1
@@
 F 2 "Custom:GP2S60_ReverseMount" H 7750 4050 50  0001 C CNN
 F 3 "" H 7750 4050 50  0001 C CNN
+F 4 "C83485" H 7750 4050 50  0001 C CNN "LCSC"
+F 5 "GP2S60B" H 7750 4050 50  0001 C CNN "Manufacturer Nbr"
 	1    7750 4050
 	1    0    0    -1
@@
 F 2 "Resistor_SMD:R_0805_2012Metric" V 7880 3300 50  0001 C CNN
 F 3 "~" H 7950 3300 50  0001 C CNN
+F 4 "C25281" H 7950 3300 50  0001 C CNN "LCSC"
+F 5 "0805W8J0120T5E" H 7950 3300 50  0001 C CNN "Manufacturer Nbr"
 	1    7950 3300
 	1    0    0    -1
@@
 F 2 "Resistor_SMD:R_0805_2012Metric" V 7480 3300 50  0001 C CNN
 F 3 "~" H 7550 3300 50  0001 C CNN
+F 4 "C38522" H 7550 3300 50  0001 C CNN "LCSC"
+F 5 "0805W8F1002T5E" H 7550 3300 50  0001 C CNN "Manufacturer Nbr"
 	1    7550 3300
 	1    0    0    -1
@@
 F 2 "Custom:GP2S60_ReverseMount" H 9550 4050 50  0001 C CNN
 F 3 "" H 9550 4050 50  0001 C CNN
+F 4 "C83485" H 9550 4050 50  0001 C CNN "LCSC"
+F 5 "GP2S60B" H 9550 4050 50  0001 C CNN "Manufacturer Nbr"
 	1    9550 4050
-	1    0    0    -1
-$EndComp
-$Comp
-L power:GND #PWR?
-U 1 1 5D73E214
-P 9550 4600
-AR Path="/5D63B6F4/5D73E214" Ref="#PWR?"  Part="1"
-AR Path="/5D63FA00/5D73E214" Ref="#PWR?"  Part="1"
-AR Path="/5D73E214" Ref="#PWR04"  Part="1"
-F 0 "#PWR04" H 9550 4350 50  0001 C CNN
-F 1 "GND" H 9555 4427 50  0000 C CNN
-F 2 "" H 9550 4600 50  0001 C CNN
-F 3 "" H 9550 4600 50  0001 C CNN
-	1    9550 4600
 	1    0    0    -1
 $EndComp
@@
 F 2 "Resistor_SMD:R_0805_2012Metric" V 9680 3300 50  0001 C CNN
 F 3 "~" H 9750 3300 50  0001 C CNN
+F 4 "C25281" H 9750 3300 50  0001 C CNN "LCSC"
+F 5 "0805W8J0120T5E" H 9750 3300 50  0001 C CNN "Manufacturer Nbr"
 	1    9750 3300
 	1    0    0    -1
@@
 F 2 "Resistor_SMD:R_0805_2012Metric" V 9280 3300 50  0001 C CNN
 F 3 "~" H 9350 3300 50  0001 C CNN
+F 4 "C38522" H 9350 3300 50  0001 C CNN "LCSC"
+F 5 "0805W8F1002T5E" H 9350 3300 50  0001 C CNN "Manufacturer Nbr"
 	1    9350 3300
 	1    0    0    -1
@@
 P 6200 1650
 F 0 "H11" H 6112 1490 50  0000 R CNN
-F 1 "M_~SLP" H 6112 1588 50  0000 R CNN
+F 1 "M~SLP" H 6112 1588 50  0000 R CNN
 F 2 "Custom:Mounting_Pad_Signal" H 6200 1800 50  0001 C CNN
 F 3 "" H 6200 1800 50  0001 C CNN
@@
 Wire Wire Line
 	5000 7350 5000 7450
-Text Notes 8550 5000 0    50   ~ 0
-Assembly
 $Comp
 L Custom:MountingPad H20
@@
 	9500 2000 9500 2100
 $Comp
-L Connector_Generic:Conn_01x02 J1
-U 1 1 5D98AE31
-P 8750 5450
-F 0 "J1" V 8622 5530 50  0000 L CNN
-F 1 "Conn_01x02" V 8713 5530 50  0000 L CNN
-F 2 "Custom:BG300-02-A-L-A" H 8750 5450 50  0001 C CNN
-F 3 "~" H 8750 5450 50  0001 C CNN
-	1    8750 5450
-	0    1    1    0
-$EndComp
-NoConn ~ 8750 5250
-NoConn ~ 8650 5250
+L power:GND #PWR?
+U 1 1 5D73E214
+P 9550 4600
+AR Path="/5D63B6F4/5D73E214" Ref="#PWR?"  Part="1"
+AR Path="/5D63FA00/5D73E214" Ref="#PWR?"  Part="1"
+AR Path="/5D73E214" Ref="#PWR04"  Part="1"
+F 0 "#PWR04" H 9550 4350 50  0001 C CNN
+F 1 "GND" H 9555 4427 50  0000 C CNN
+F 2 "" H 9550 4600 50  0001 C CNN
+F 3 "" H 9550 4600 50  0001 C CNN
+	1    9550 4600
+	1    0    0    -1
+$EndComp
 $EndSCHEMATC
