File: robot/Side/Side/Side.kicad_pcb (KiCad board)
At the start: 2 copper layers, 40 x 40 mm, 3 parts, among them J1 Conn_01x01

Commit message: Small changes, connectors
Parts:
- added H3: GND, Custom:Mounting_Pad_Power, F.Cu at (177.4, 76.2)
- added H4: GND, Custom:Mounting_Pad_Power, B.Cu at (177.4, 76.2)
- added H5: GND, Custom:Mounting_Pad_Power_Corner, F.Cu at (213.8, 111.3)
- added H6: GND, Custom:Mounting_Pad_Power_Corner, B.Cu at (213.8, 78.7)
- added H7: GND, Custom:Mounting_Pad_Power_Corner, F.Cu at (211.3, 76.2)
- added H8: GND, Custom:Mounting_Pad_Power_Corner, B.Cu at (211.3, 113.8)
- added J2: Conn_01x02, Custom:BG300-02-A-L-A, B.Cu at (190.4, 95.0)
- added J3: Conn_01x02, Custom:BG300-02-A-L-A, F.Cu at (190.4, 95.0)
- moved H1 35.1 mm to (177.4, 113.8)
- moved H2 35.1 mm to (177.4, 113.8)
Routing:
- net GND: track 0.00 -> 9.73 mm, vias 2 -> 8
Other:
- net class Power added: clearance 0.2, trace_width 0.3, via_dia 0.8, via_drill 0.4
Changed lines of the file:
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@@
     (thickness 1.6)
     (drawings 8)
-    (tracks 2)
+    (tracks 13)
     (zones 0)
-    (modules 3)
+    (modules 11)
     (nets 3)
   )
@@
     (uvia_dia 0.3)
     (uvia_drill 0.1)
+  )
+  (net_class Power ""
+    (clearance 0.2)
+    (trace_width 0.3)
+    (via_dia 0.8)
+    (via_drill 0.4)
+    (uvia_dia 0.3)
+    (uvia_drill 0.1)
     (add_net /VBUS)
     (add_net GND)
+  )
+  (module Custom:BG300-02-A-L-A (layer B.Cu)
+    (at 190.39 95 90)
+    (fp_text reference J2 (at 0 -12.5 90) (layer B.Fab)
+      (effects (font (size 1 1) (thickness 0.15)) (justify mirror))
+    )
+    (fp_text value Conn_01x02 (at 0 0.5 90) (layer B.Fab)
+      (effects (font (size 1 1) (thickness 0.15)) (justify mirror))
+    )
+    (fp_line (start -2.83 -11.5) (end -2.83 -3) (layer B.Fab) (width 0.12))
+    (fp_line (start 2.82 -11.5) (end -2.83 -11.5) (layer B.Fab) (width 0.12))
+    (fp_line (start 2.82 -3) (end 2.82 -11.5) (layer B.Fab) (width 0.12))
+    (fp_line (start -2.83 -3) (end 2.82 -3) (layer B.Fab) (width 0.12))
+    (pad 2 smd rect (at 1.26 -1.5 90) (size 1 2) (layers B.Cu B.Paste B.Mask)
+      (net 2 GND))
+    (pad 1 smd rect (at -1.26 -1.5 90) (size 1 2) (layers B.Cu B.Paste B.Mask)
+      (net 2 GND))
+  )
+  (module Custom:BG300-02-A-L-A (layer F.Cu)
+    (at 190.39 95 270)
+    (fp_text reference J3 (at 0 12.5 90) (layer F.Fab)
+      (effects (font (size 1 1) (thickness 0.15)))
+    )
+    (fp_text value Conn_01x02 (at 0 -0.5 90) (layer F.Fab)
+      (effects (font (size 1 1) (thickness 0.15)))
+    )
+    (fp_line (start -2.83 11.5) (end -2.83 3) (layer F.Fab) (width 0.12))
+    (fp_line (start 2.82 11.5) (end -2.83 11.5) (layer F.Fab) (width 0.12))
+    (fp_line (start 2.82 3) (end 2.82 11.5) (layer F.Fab) (width 0.12))
+    (fp_line (start -2.83 3) (end 2.82 3) (layer F.Fab) (width 0.12))
+    (pad 2 smd rect (at 1.26 1.5 270) (size 1 2) (layers F.Cu F.Paste F.Mask)
+      (net 2 GND))
+    (pad 1 smd rect (at -1.26 1.5 270) (size 1 2) (layers F.Cu F.Paste F.Mask)
+      (net 2 GND))
   )
   (module Custom:Axis (layer F.Cu)
@@
   )
   (module Custom:Mounting_Pad_Power (layer B.Cu)
-    (at 212.525 113.775 90)
+    (at 177.45 113.8 90)
     (fp_text reference H1 (at 0.25 -3.425 90) (layer B.Fab)
       (effects (font (size 1 1) (thickness 0.15)) (justify mirror))
@@
   )
   (module Custom:Mounting_Pad_Power (layer F.Cu)
-    (at 212.525 113.775 90)
+    (at 177.45 113.8 90)
     (fp_text reference H2 (at 0 3.9 90) (layer F.Fab)
       (effects (font (size 1 1) (thickness 0.15)))
@@
       (net 2 GND))
   )
-  (gr_line (start 215 88.4) (end 215 115) (layer Edge.Cuts) (width 0.05))
-  (gr_line (start 212.5 88.4) (end 215 88.4) (layer Edge.Cuts) (width 0.05))
-  (gr_line (start 212.5 80.9) (end 212.5 88.4) (layer Edge.Cuts) (width 0.05))
-  (gr_line (start 215 80.9) (end 212.5 80.9) (layer Edge.Cuts) (width 0.05))
-  (gr_line (start 215 75) (end 215 80.9) (layer Edge.Cuts) (width 0.05))
-  (gr_line (start 175 115) (end 175 75) (layer Edge.Cuts) (width 0.05))
-  (gr_line (start 215 115) (end 175 115) (layer Edge.Cuts) (width 0.05))
-  (gr_line (start 175 75) (end 215 75) (layer Edge.Cuts) (width 0.05))
-  (via (at 213.75 113.75) (size 0.8) (drill 0.4) (layers F.Cu B.Cu) (net 2))
-  (via (at 211.25 113.75) (size 0.8) (drill 0.4) (layers F.Cu B.Cu) (net 2))
+  (module Custom:Mounting_Pad_Power (layer F.Cu)
+    (at 177.45 76.2 270)
+    (fp_text reference H3 (at 0 3.9 90) (layer F.Fab)
+      (effects (font (size 1 1) (thickness 0.15)))
+    )
+    (fp_text value GND (at 0 -4.1 90) (layer F.Fab)
+      (effects (font (size 1 1) (thickness 0.15)))
+    )
+    (pad 1 smd rect (at 0 0 270) (size 2.5 5) (layers F.Cu F.Paste F.Mask)
+      (net 2 GND))
+  )
+  (module Custom:Mounting_Pad_Power (layer B.Cu)
+    (at 177.45 76.2 90)
+    (fp_text reference H4 (at 0 -3.9 90) (layer B.Fab)
+      (effects (font (size 1 1) (thickness 0.15)) (justify mirror))
+    )
+    (fp_text value GND (at 0 4.1 90) (layer B.Fab)
+      (effects (font (size 1 1) (thickness 0.15)) (justify mirror))
+    )
+    (pad 1 smd rect (at 0 0 90) (size 2.5 5) (layers B.Cu B.Paste B.Mask)
+      (net 2 GND))
+  )
+  (module Custom:Mounting_Pad_Power_Corner (layer F.Cu)
+    (at 213.8 111.3 270)
+    (fp_text reference H5 (at 0 3.9 90) (layer F.Fab)
+      (effects (font (size 1 1) (thickness 0.15)))
+    )
+    (fp_text value GND (at -2 1.27 90) (layer F.Fab)
+      (effects (font (size 1 1) (thickness 0.15)))
+    )
+    (pad 1 smd custom (at 0 0 270) (size 2.5 2.5) (layers F.Cu F.Paste F.Mask)
+      (net 2 GND) (zone_connect 0)
+      (options (clearance outline) (anchor rect))
+      (primitives
+        (gr_poly (pts
+           (xy 1.25 -1.25) (xy 3.75 -1.25) (xy 3.75 3.75) (xy 1.25 3.75) (xy 1.25 1.25)
+           (xy -1.25 1.25) (xy -1.25 -1.25) (xy 1.244445 -1.25)) (width 0))
+      ))
+  )
+  (module Custom:Mounting_Pad_Power_Corner (layer B.Cu)
+    (at 213.8 78.7 90)
+    (fp_text reference H6 (at 0 -3.9 90) (layer B.Fab)
+      (effects (font (size 1 1) (thickness 0.15)) (justify mirror))
+    )
+    (fp_text value GND (at 0.49 -3.74 90) (layer B.Fab)
+      (effects (font (size 1 1) (thickness 0.15)) (justify mirror))
+    )
+    (pad 1 smd custom (at 0 0 90) (size 2.5 2.5) (layers B.Cu B.Paste B.Mask)
+      (net 2 GND) (zone_connect 0)
+      (options (clearance outline) (anchor rect))
+      (primitives
+        (gr_poly (pts
+           (xy 1.25 1.25) (xy 3.75 1.25) (xy 3.75 -3.75) (xy 1.25 -3.75) (xy 1.25 -1.25)
+           (xy -1.25 -1.25) (xy -1.25 1.25) (xy 1.244445 1.25)) (width 0))
+      ))
+  )
+  (module Custom:Mounting_Pad_Power_Corner (layer F.Cu)
+    (at 211.3 76.2)
+    (fp_text reference H7 (at 0 3.9) (layer F.Fab)
+      (effects (font (size 1 1) (thickness 0.15)))
+    )
+    (fp_text value GND (at -2.63 1.86) (layer F.Fab)
+      (effects (font (size 1 1) (thickness 0.15)))
+    )
+    (pad 1 smd custom (at 0 0) (size 2.5 2.5) (layers F.Cu F.Paste F.Mask)
+      (net 2 GND) (zone_connect 0)
+      (options (clearance outline) (anchor rect))
+      (primitives
+        (gr_poly (pts
+           (xy 1.25 -1.25) (xy 3.75 -1.25) (xy 3.75 3.75) (xy 1.25 3.75) (xy 1.25 1.25)
+           (xy -1.25 1.25) (xy -1.25 -1.25) (xy 1.244445 -1.25)) (width 0))
+      ))
+  )
+  (module Custom:Mounting_Pad_Power_Corner (layer B.Cu)
+    (at 211.3 113.8)
+    (fp_text reference H8 (at 0 -3.9) (layer B.Fab)
+      (effects (font (size 1 1) (thickness 0.15)) (justify mirror))
+    )
+    (fp_text value GND (at -2.54 -1.3) (layer B.Fab)
+      (effects (font (size 1 1) (thickness 0.15)) (justify mirror))
+    )
+    (pad 1 smd custom (at 0 0) (size 2.5 2.5) (layers B.Cu B.Paste B.Mask)
+      (net 2 GND) (zone_connect 0)
+      (options (clearance outline) (anchor rect))
+      (primitives
+        (gr_poly (pts
+           (xy 1.25 1.25) (xy 3.75 1.25) (xy 3.75 -3.75) (xy 1.25 -3.75) (xy 1.25 -1.25)
+           (xy -1.25 -1.25) (xy -1.25 1.25) (xy 1.244445 1.25)) (width 0))
+      ))
+  )
+  (gr_line (start 215 75) (end 215 80.9) (layer Edge.Cuts) (width 0.1))
+  (gr_line (start 215 88.4) (end 215 115) (layer Edge.Cuts) (width 0.1))
+  (gr_line (start 212.5 88.4) (end 215 88.4) (layer Edge.Cuts) (width 0.1))
+  (gr_line (start 212.5 80.9) (end 212.5 88.4) (layer Edge.Cuts) (width 0.1))
+  (gr_line (start 215 80.9) (end 212.5 80.9) (layer Edge.Cuts) (width 0.1))
+  (gr_line (start 175 115) (end 175 75) (layer Edge.Cuts) (width 0.1))
+  (gr_line (start 215 115) (end 175 115) (layer Edge.Cuts) (width 0.1))
+  (gr_line (start 175 75) (end 215 75) (layer Edge.Cuts) (width 0.1))
+  (via (at 177.45 76.2) (size 0.8) (drill 0.4) (layers F.Cu B.Cu) (net 2))
+  (via (at 177.45 113.8) (size 0.8) (drill 0.4) (layers F.Cu B.Cu) (net 2))
+  (via (at 211.3 76.2) (size 0.8) (drill 0.4) (layers F.Cu B.Cu) (net 2))
+  (via (at 213.8 78.7) (size 0.8) (drill 0.4) (layers F.Cu B.Cu) (net 2))
+  (segment (start 213.8 78.7) (end 211.37 78.7) (width 0.3) (layer B.Cu) (net 2))
+  (segment (start 211.3 76.2) (end 211.3 77.55) (width 0.3) (layer F.Cu) (net 2))
+  (segment (start 211.3 77.55) (end 211.3 78.63) (width 0.3) (layer F.Cu) (net 2))
+  (via (at 211.3 113.8) (size 0.8) (drill 0.4) (layers F.Cu B.Cu) (net 2))
+  (segment (start 211.3 113.8) (end 211.3 111.43) (width 0.3) (layer B.Cu) (net 2))
+  (via (at 213.8 111.3) (size 0.8) (drill 0.4) (layers F.Cu B.Cu) (net 2))
+  (segment (start 213.8 111.3) (end 211.3 111.3) (width 0.3) (layer F.Cu) (net 2))
+  (via (at 188.89 93.74) (size 0.8) (drill 0.4) (layers F.Cu B.Cu) (net 2))
+  (via (at 188.89 96.26) (size 0.8) (drill 0.4) (layers F.Cu B.Cu) (net 2))
   (zone (net 2) (net_name GND) (layer F.Cu) (hatch edge 0.508)
     (connect_pads (clearance 0.508))
