File: robot/Side/Side/Side.sch (KiCad schematic (older format))
At the start: 3 parts, among them J1 Conn_01x01

Commit message: Small changes, connectors
Parts:
- added H3, H4: GND, Custom:Mounting_Pad_Power, symbol Custom:MountingPad
- added H5, H6, H7, H8: GND, Custom:Mounting_Pad_Power_Corner, symbol Custom:MountingPad
- added J2, J3: Conn_01x02, Custom:BG300-02-A-L-A, symbol Connector_Generic:Conn_01x02
Connections:
- net GND: now also H3.1 (Pin), H4.1 (Pin), H5.1 (Pin), H6.1 (Pin), H7.1 (Pin), H8.1 (Pin), J2.1 (Pin_1), J2.2 (Pin_2), J3.1 (Pin_1), J3.2 (Pin_2)
Other:
- note added: "Corners"
Changed lines of the file:
@@
 	1    0    0    -1
 $EndComp
+$Comp
+L Custom:MountingPad H3
+U 1 1 5D9BF32E
+P 2800 3650
+F 0 "H3" H 2600 3600 50  0000 L CNN
+F 1 "GND" H 2550 3500 50  0000 L CNN
+F 2 "Custom:Mounting_Pad_Power" H 2800 3800 50  0001 C CNN
+F 3 "" H 2800 3800 50  0001 C CNN
+	1    2800 3650
+	1    0    0    -1
+$EndComp
+$Comp
+L power:GND #PWR0104
+U 1 1 5D9BF338
+P 2800 4000
+F 0 "#PWR0104" H 2800 3750 50  0001 C CNN
+F 1 "GND" H 2805 3827 50  0000 C CNN
+F 2 "" H 2800 4000 50  0001 C CNN
+F 3 "" H 2800 4000 50  0001 C CNN
+	1    2800 4000
+	1    0    0    -1
+$EndComp
+Wire Wire Line
+	2800 3950 2800 4000
+Wire Wire Line
+	2800 5850 2800 5900
+$Comp
+L power:GND #PWR0105
+U 1 1 5D9BF975
+P 2800 5900
+F 0 "#PWR0105" H 2800 5650 50  0001 C CNN
+F 1 "GND" H 2805 5727 50  0000 C CNN
+F 2 "" H 2800 5900 50  0001 C CNN
+F 3 "" H 2800 5900 50  0001 C CNN
+	1    2800 5900
+	1    0    0    -1
+$EndComp
+$Comp
+L Custom:MountingPad H5
+U 1 1 5D9BF97F
+P 2800 5550
+F 0 "H5" H 2888 5488 50  0000 L CNN
+F 1 "GND" H 2888 5397 50  0000 L CNN
+F 2 "Custom:Mounting_Pad_Power_Corner" H 2800 5700 50  0001 C CNN
+F 3 "" H 2800 5700 50  0001 C CNN
+	1    2800 5550
+	1    0    0    -1
+$EndComp
+$Comp
+L Custom:MountingPad H4
+U 1 1 5D9C022F
+P 3400 3650
+F 0 "H4" H 3200 3600 50  0000 L CNN
+F 1 "GND" H 3150 3500 50  0000 L CNN
+F 2 "Custom:Mounting_Pad_Power" H 3400 3800 50  0001 C CNN
+F 3 "" H 3400 3800 50  0001 C CNN
+	1    3400 3650
+	1    0    0    -1
+$EndComp
+$Comp
+L power:GND #PWR0106
+U 1 1 5D9C0239
+P 3400 4000
+F 0 "#PWR0106" H 3400 3750 50  0001 C CNN
+F 1 "GND" H 3405 3827 50  0000 C CNN
+F 2 "" H 3400 4000 50  0001 C CNN
+F 3 "" H 3400 4000 50  0001 C CNN
+	1    3400 4000
+	1    0    0    -1
+$EndComp
+Wire Wire Line
+	3400 3950 3400 4000
+Wire Wire Line
+	2800 6600 2800 6650
+$Comp
+L power:GND #PWR0107
+U 1 1 5D9C0245
+P 2800 6650
+F 0 "#PWR0107" H 2800 6400 50  0001 C CNN
+F 1 "GND" H 2805 6477 50  0000 C CNN
+F 2 "" H 2800 6650 50  0001 C CNN
+F 3 "" H 2800 6650 50  0001 C CNN
+	1    2800 6650
+	1    0    0    -1
+$EndComp
+$Comp
+L Custom:MountingPad H6
+U 1 1 5D9C024F
+P 2800 6300
+F 0 "H6" H 2888 6238 50  0000 L CNN
+F 1 "GND" H 2888 6147 50  0000 L CNN
+F 2 "Custom:Mounting_Pad_Power_Corner" H 2800 6450 50  0001 C CNN
+F 3 "" H 2800 6450 50  0001 C CNN
+	1    2800 6300
+	1    0    0    -1
+$EndComp
+Wire Wire Line
+	3350 5850 3350 5900
+$Comp
+L power:GND #PWR0108
+U 1 1 5D9C4095
+P 3350 5900
+F 0 "#PWR0108" H 3350 5650 50  0001 C CNN
+F 1 "GND" H 3355 5727 50  0000 C CNN
+F 2 "" H 3350 5900 50  0001 C CNN
+F 3 "" H 3350 5900 50  0001 C CNN
+	1    3350 5900
+	1    0    0    -1
+$EndComp
+$Comp
+L Custom:MountingPad H7
+U 1 1 5D9C409F
+P 3350 5550
+F 0 "H7" H 3438 5488 50  0000 L CNN
+F 1 "GND" H 3438 5397 50  0000 L CNN
+F 2 "Custom:Mounting_Pad_Power_Corner" H 3350 5700 50  0001 C CNN
+F 3 "" H 3350 5700 50  0001 C CNN
+	1    3350 5550
+	1    0    0    -1
+$EndComp
+Wire Wire Line
+	3350 6600 3350 6650
+$Comp
+L power:GND #PWR0109
+U 1 1 5D9C40AA
+P 3350 6650
+F 0 "#PWR0109" H 3350 6400 50  0001 C CNN
+F 1 "GND" H 3355 6477 50  0000 C CNN
+F 2 "" H 3350 6650 50  0001 C CNN
+F 3 "" H 3350 6650 50  0001 C CNN
+	1    3350 6650
+	1    0    0    -1
+$EndComp
+$Comp
+L Custom:MountingPad H8
+U 1 1 5D9C40B4
+P 3350 6300
+F 0 "H8" H 3438 6238 50  0000 L CNN
+F 1 "GND" H 3438 6147 50  0000 L CNN
+F 2 "Custom:Mounting_Pad_Power_Corner" H 3350 6450 50  0001 C CNN
+F 3 "" H 3350 6450 50  0001 C CNN
+	1    3350 6300
+	1    0    0    -1
+$EndComp
+Text Notes 2950 5250 0    50   ~ 0
+Corners
+$Comp
+L Connector_Generic:Conn_01x02 J3
+U 1 1 5D9BA9E9
+P 3100 1950
+F 0 "J3" H 3180 1942 50  0000 L CNN
+F 1 "Conn_01x02" H 3180 1851 50  0000 L CNN
+F 2 "Custom:BG300-02-A-L-A" H 3100 1950 50  0001 C CNN
+F 3 "~" H 3100 1950 50  0001 C CNN
+	1    3100 1950
+	1    0    0    -1
+$EndComp
+$Comp
+L Connector_Generic:Conn_01x02 J2
+U 1 1 5D9BC21F
+P 3100 1400
+F 0 "J2" H 3180 1392 50  0000 L CNN
+F 1 "Conn_01x02" H 3180 1301 50  0000 L CNN
+F 2 "Custom:BG300-02-A-L-A" H 3100 1400 50  0001 C CNN
+F 3 "~" H 3100 1400 50  0001 C CNN
+	1    3100 1400
+	1    0    0    -1
+$EndComp
+$Comp
+L power:GND #PWR?
+U 1 1 5D9BF453
+P 2700 1500
+F 0 "#PWR?" H 2700 1250 50  0001 C CNN
+F 1 "GND" H 2705 1327 50  0000 C CNN
+F 2 "" H 2700 1500 50  0001 C CNN
+F 3 "" H 2700 1500 50  0001 C CNN
+	1    2700 1500
+	1    0    0    -1
+$EndComp
+Wire Wire Line
+	2800 1400 2900 1400
+Wire Wire Line
+	2800 1500 2900 1500
+Wire Wire Line
+	2800 1950 2900 1950
+Wire Wire Line
+	2800 2050 2900 2050
+$Comp
+L power:GND #PWR?
+U 1 1 5D9BEA51
+P 2700 2050
+F 0 "#PWR?" H 2700 1800 50  0001 C CNN
+F 1 "GND" H 2705 1877 50  0000 C CNN
+F 2 "" H 2700 2050 50  0001 C CNN
+F 3 "" H 2700 2050 50  0001 C CNN
+	1    2700 2050
+	1    0    0    -1
+$EndComp
+Wire Wire Line
+	2800 1950 2800 2000
+Wire Wire Line
+	2800 1400 2800 1450
+Wire Wire Line
+	2800 1450 2700 1450
+Wire Wire Line
+	2700 1450 2700 1500
+Connection ~ 2800 1450
+Wire Wire Line
+	2800 1450 2800 1500
+Wire Wire Line
+	2800 2000 2700 2000
+Wire Wire Line
+	2700 2000 2700 2050
+Connection ~ 2800 2000
+Wire Wire Line
+	2800 2000 2800 2050
 $EndSCHEMATC
